File: usb-solder/usb-solder.kicad_pcb (KiCad board)
At the start: 2 copper layers, 100 x 100 mm, 187 parts, among them J1 USB_B_Micro, J10 USB_B_Micro, J11 USB_B_Micro, J12 USB_B_Micro, J13 USB_B_Micro, J14 USB_B_Micro, J15 USB_B_Micro, J16 USB_B_Micro, J17 USB_B_Micro, J18 USB_B_Micro, J19 Barrel_Jack_Switch, J2 USB_B_Micro, J20 Conn_01x02_Male, J21 USB_B_Micro, J22 USB_B_Micro, J23 USB_B_Micro, J24 USB_A, J25 USB_B_Micro, J26 USB_B_Micro, J27 USB_B_Micro, J3 USB_B_Micro, J4 USB_B_Micro, J5 USB_B_Micro, J6 USB_B_Micro, J7 USB_B_Micro, J8 USB_B_Micro, J9 USB_B_Micro, U1 555, U2 74HC164, U3 4072, U4 74HC04, U5 AP1117-33

Commit message: new
Parts:
- removed the D113 at (284.0, 55.3)
- removed D115, D116, D117, D118, D120, D121, D122, D123, D124, D125, D126, D128, D129, D130, D131, D132, D133, D134, D136, D137, D138, D139, D140, D141, D142, D144, D145: ledred, LED_SMD:LED_0603_1608Metric
- removed the J22 at (147.3, 100.2)
- removed the J23 at (147.3, 89.2)
- removed the J25 at (147.3, 78.3)
- removed the J3 at (52.7, 78.4)
- added C5: 100n, Capacitor_SMD:C_0402_1005Metric, F.Cu at (166.4, 67.4)
- added D102: ledred, LED_SMD:LED_0603_1608Metric, F.Cu at (160.1, 56.1)
- added D109: ledred, LED_SMD:LED_0603_1608Metric, F.Cu at (181.6, 40.6)
- added D111: ledred, LED_SMD:LED_0603_1608Metric, F.Cu at (193.8, 27.5)
- added D43: ledred, LED_SMD:LED_0603_1608Metric, F.Cu at (168.4, 37.4)
- added D84: ledred, LED_SMD:LED_0603_1608Metric, F.Cu at (162.4, 61.2)
- added H1: MountingHole, MountingHole:MountingHole_3.5mm, F.Cu at (53.8, 53.7)
- added H2: MountingHole, MountingHole:MountingHole_3.5mm, F.Cu at (146.3, 146.3)
- added H3: MountingHole, MountingHole:MountingHole_3.5mm, F.Cu at (53.7, 146.3)
- added H4: MountingHole, MountingHole:MountingHole_3.5mm, F.Cu at (146.3, 53.7)
- added J1: USB_B_Micro, Connector_USB:USB_Micro-B_Molex-105017-0001, F.Cu at (51.8, 61.9)
- added J19: USB_B_Micro, Connector_USB:USB_Micro-B_Molex-105017-0001, F.Cu at (146.7, 87.3)
- added J20: USB_B_Micro, Connector_USB:USB_Micro-B_Molex-105017-0001, F.Cu at (160.8, 23.4)
- added R3: 10k, Resistor_SMD:R_0402_1005Metric, F.Cu at (181.0, 67.3)
- added R4: 10k, Resistor_SMD:R_0402_1005Metric, F.Cu at (178.1, 67.3)
- added R5: 10k, Resistor_SMD:R_0402_1005Metric, F.Cu at (175.2, 67.9)
- added R6: 10k, Resistor_SMD:R_0402_1005Metric, F.Cu at (172.2, 67.9)
- added R7: 10k, Resistor_SMD:R_0402_1005Metric, F.Cu at (169.3, 67.9)
- added R8: 10k, Resistor_SMD:R_0402_1005Metric, F.Cu at (164.8, 64.5)
- added R9: 10k, Resistor_SMD:R_0402_1005Metric, F.Cu at (153.2, 68.1)
- added SW1: SW_SPDT, pace:Switch_Toggle_ATE1D-2M3-10-Z, F.Cu at (127.2, 36.4)
- added TP1: TestPoint, TestPoint:TestPoint_Pad_D1.0mm, F.Cu at (188.1, 38.8)
- added TP10: TestPoint, TestPoint:TestPoint_Pad_D1.0mm, F.Cu at (209.9, 14.7)
- added TP100: TestPoint, TestPoint:TestPoint_Pad_D1.0mm, F.Cu at (181.1, 64.7)
- added TP101: TestPoint, TestPoint:TestPoint_Pad_D1.0mm, F.Cu at (218.7, 26.9)
- added TP102: TestPoint, TestPoint:TestPoint_Pad_D1.0mm, F.Cu at (215.6, 30.0)
- added TP103: TestPoint, TestPoint:TestPoint_Pad_D1.0mm, F.Cu at (203.4, 41.3)
- added TP104: TestPoint, TestPoint:TestPoint_Pad_D1.0mm, F.Cu at (200.3, 43.4)
- added TP105: TestPoint, TestPoint:TestPoint_Pad_D1.0mm, F.Cu at (209.9, 36.1)
- added TP106: TestPoint, TestPoint:TestPoint_Pad_D1.0mm, F.Cu at (212.9, 33.0)
- added TP107: TestPoint, TestPoint:TestPoint_Pad_D1.0mm, F.Cu at (163.4, 67.1)
- added TP108: TestPoint, TestPoint:TestPoint_Pad_D1.0mm, F.Cu at (198.4, 46.5)
- added TP109: TestPoint, TestPoint:TestPoint_Pad_D1.0mm, F.Cu at (196.1, 51.2)
- added TP11: TestPoint, TestPoint:TestPoint_Pad_D1.0mm, F.Cu at (194.2, 39.0)
- added TP110: TestPoint, TestPoint:TestPoint_Pad_D1.0mm, F.Cu at (190.3, 57.3)
- added TP111: TestPoint, TestPoint:TestPoint_Pad_D1.0mm, F.Cu at (193.3, 54.2)
- added TP112: TestPoint, TestPoint:TestPoint_Pad_D1.0mm, F.Cu at (187.2, 60.3)
- added TP113: TestPoint, TestPoint:TestPoint_Pad_D1.0mm, F.Cu at (186.9, 51.2)
- added TP114: TestPoint, TestPoint:TestPoint_Pad_D1.0mm, F.Cu at (191.2, 39.0)
- added TP115: TestPoint, TestPoint:TestPoint_Pad_D1.0mm, F.Cu at (194.6, 35.9)
- added TP117: TestPoint, TestPoint:TestPoint_Pad_D1.0mm, F.Cu at (203.8, 35.2)
- added TP118: TestPoint, TestPoint:TestPoint_Pad_D1.0mm, F.Cu at (206.8, 33.0)
- added TP119: TestPoint, TestPoint:TestPoint_Pad_D1.0mm, F.Cu at (196.4, 54.2)
- added TP12: TestPoint, TestPoint:TestPoint_Pad_D1.0mm, F.Cu at (184.1, 44.9)
- added TP120: TestPoint, TestPoint:TestPoint_Pad_D1.0mm, F.Cu at (218.7, 30.0)
- added TP121: TestPoint, TestPoint:TestPoint_Pad_D1.0mm, F.Cu at (184.2, 64.7)
- added TP122: TestPoint, TestPoint:TestPoint_Pad_D1.0mm, F.Cu at (209.9, 39.1)
- added TP123: TestPoint, TestPoint:TestPoint_Pad_D1.0mm, F.Cu at (212.9, 36.1)
- added TP124: TestPoint, TestPoint:TestPoint_Pad_D1.0mm, F.Cu at (190.3, 54.2)
- added TP125: TestPoint, TestPoint:TestPoint_Pad_D1.0mm, F.Cu at (206.4, 42.2)
- added TP126: TestPoint, TestPoint:TestPoint_Pad_D1.0mm, F.Cu at (199.1, 49.5)
- added TP127: TestPoint, TestPoint:TestPoint_Pad_D1.0mm, F.Cu at (190.3, 60.3)
- added TP129: TestPoint, TestPoint:TestPoint_Pad_D1.0mm, F.Cu at (201.4, 46.5)
- added TP13: TestPoint, TestPoint:TestPoint_Pad_D1.0mm, F.Cu at (188.1, 41.9)
- added TP130: TestPoint, TestPoint:TestPoint_Pad_D1.0mm, F.Cu at (184.2, 61.7)
- added TP131: TestPoint, TestPoint:TestPoint_Pad_D1.0mm, F.Cu at (195.3, 48.1)
- added TP132: TestPoint, TestPoint:TestPoint_Pad_D1.0mm, F.Cu at (193.0, 51.2)
- added TP14: TestPoint, TestPoint:TestPoint_Pad_D1.0mm, F.Cu at (200.4, 28.2)
- added TP15: TestPoint, TestPoint:TestPoint_Pad_D1.0mm, F.Cu at (160.4, 67.1)
- added TP16: TestPoint, TestPoint:TestPoint_Pad_D1.0mm, F.Cu at (205.4, 23.0)
- added TP17: TestPoint, TestPoint:TestPoint_Pad_D1.0mm, F.Cu at (191.6, 35.9)
- added TP19: TestPoint, TestPoint:TestPoint_Pad_D1.0mm, F.Cu at (174.7, 53.1)
- added TP2: TestPoint, TestPoint:TestPoint_Pad_D1.0mm, F.Cu at (165.9, 58.9)
- added TP20: TestPoint, TestPoint:TestPoint_Pad_D1.0mm, F.Cu at (181.1, 46.4)
- added TP21: TestPoint, TestPoint:TestPoint_Pad_D1.0mm, F.Cu at (209.9, 17.8)
- added TP22: TestPoint, TestPoint:TestPoint_Pad_D1.0mm, F.Cu at (213.0, 14.7)
- added TP23: TestPoint, TestPoint:TestPoint_Pad_D1.0mm, F.Cu at (185.1, 38.8)
- added TP24: TestPoint, TestPoint:TestPoint_Pad_D1.0mm, F.Cu at (188.5, 35.5)
- added TP25: TestPoint, TestPoint:TestPoint_Pad_D1.0mm, F.Cu at (171.7, 53.1)
- added TP26: TestPoint, TestPoint:TestPoint_Pad_D1.0mm, F.Cu at (157.3, 66.7)
- added TP27: TestPoint, TestPoint:TestPoint_Pad_D1.0mm, F.Cu at (197.7, 37.3)
- added TP28: TestPoint, TestPoint:TestPoint_Pad_D1.0mm, F.Cu at (57.0, 141.5)
- added TP29: TestPoint, TestPoint:TestPoint_Pad_D1.0mm, F.Cu at (172.0, 56.2)
- added TP3: TestPoint, TestPoint:TestPoint_Pad_D1.0mm, F.Cu at (197.3, 27.7)
- added TP30: TestPoint, TestPoint:TestPoint_Pad_D1.0mm, F.Cu at (213.0, 17.8)
- added TP31: TestPoint, TestPoint:TestPoint_Pad_D1.0mm, F.Cu at (208.9, 20.8)
- added TP32: TestPoint, TestPoint:TestPoint_Pad_D1.0mm, F.Cu at (216.0, 14.7)
- added TP33: TestPoint, TestPoint:TestPoint_Pad_D1.0mm, F.Cu at (177.8, 52.5)
- added TP34: TestPoint, TestPoint:TestPoint_Pad_D1.0mm, F.Cu at (204.4, 26.0)
- added TP35: TestPoint, TestPoint:TestPoint_Pad_D1.0mm, F.Cu at (55.4, 134.7)
- added TP36: TestPoint, TestPoint:TestPoint_Pad_D1.0mm, F.Cu at (57.0, 138.8)
- added TP37: TestPoint, TestPoint:TestPoint_Pad_D1.0mm, F.Cu at (180.1, 49.5)
- added TP38: TestPoint, TestPoint:TestPoint_Pad_D1.0mm, F.Cu at (187.2, 44.9)
- added TP39: TestPoint, TestPoint:TestPoint_Pad_D1.0mm, F.Cu at (212.0, 20.8)
- added TP4: TestPoint, TestPoint:TestPoint_Pad_D1.0mm, F.Cu at (192.6, 32.9)
- added TP41: TestPoint, TestPoint:TestPoint_Pad_D1.0mm, F.Cu at (183.1, 49.5)
- added TP42: TestPoint, TestPoint:TestPoint_Pad_D1.0mm, F.Cu at (168.9, 64.9)
- added TP43: TestPoint, TestPoint:TestPoint_Pad_D1.0mm, F.Cu at (203.4, 29.1)
- added TP44: TestPoint, TestPoint:TestPoint_Pad_D1.0mm, F.Cu at (55.4, 137.4)
- added TP45: TestPoint, TestPoint:TestPoint_Pad_D1.0mm, F.Cu at (172.0, 59.2)
- added TP46: TestPoint, TestPoint:TestPoint_Pad_D1.0mm, F.Cu at (185.1, 41.9)
- added TP47: TestPoint, TestPoint:TestPoint_Pad_D1.0mm, F.Cu at (168.9, 58.8)
- added TP48: TestPoint, TestPoint:TestPoint_Pad_D1.0mm, F.Cu at (57.0, 136.1)
- added TP49: TestPoint, TestPoint:TestPoint_Pad_D1.0mm, F.Cu at (178.1, 58.6)
- added TP5: TestPoint, TestPoint:TestPoint_Pad_D1.0mm, F.Cu at (167.6, 55.7)
- added TP50: TestPoint, TestPoint:TestPoint_Pad_D1.0mm, F.Cu at (181.1, 55.6)
- added TP51: TestPoint, TestPoint:TestPoint_Pad_D1.0mm, F.Cu at (215.0, 20.8)
- added TP52: TestPoint, TestPoint:TestPoint_Pad_D1.0mm, F.Cu at (206.5, 29.1)
- added TP53: TestPoint, TestPoint:TestPoint_Pad_D1.0mm, F.Cu at (211.5, 23.9)
- added TP54: TestPoint, TestPoint:TestPoint_Pad_D1.0mm, F.Cu at (191.2, 42.0)
- added TP55: TestPoint, TestPoint:TestPoint_Pad_D1.0mm, F.Cu at (200.7, 34.3)
- added TP56: TestPoint, TestPoint:TestPoint_Pad_D1.0mm, F.Cu at (186.2, 48.0)
- added TP57: TestPoint, TestPoint:TestPoint_Pad_D1.0mm, F.Cu at (172.0, 62.3)
- added TP58: TestPoint, TestPoint:TestPoint_Pad_D1.0mm, F.Cu at (178.1, 55.6)
- added TP6: TestPoint, TestPoint:TestPoint_Pad_D1.0mm, F.Cu at (205.9, 19.9)
- added TP60: TestPoint, TestPoint:TestPoint_Pad_D1.0mm, F.Cu at (219.1, 14.7)
- added TP61: TestPoint, TestPoint:TestPoint_Pad_D1.0mm, F.Cu at (216.0, 17.8)
- added TP62: TestPoint, TestPoint:TestPoint_Pad_D1.0mm, F.Cu at (197.7, 34.3)
- added TP63: TestPoint, TestPoint:TestPoint_Pad_D1.0mm, F.Cu at (197.3, 30.7)
- added TP64: TestPoint, TestPoint:TestPoint_Pad_D1.0mm, F.Cu at (206.8, 36.1)
- added TP65: TestPoint, TestPoint:TestPoint_Pad_D1.0mm, F.Cu at (193.3, 45.1)
- added TP66: TestPoint, TestPoint:TestPoint_Pad_D1.0mm, F.Cu at (190.2, 45.1)
- added TP67: TestPoint, TestPoint:TestPoint_Pad_D1.0mm, F.Cu at (183.9, 52.5)
- added TP68: TestPoint, TestPoint:TestPoint_Pad_D1.0mm, F.Cu at (219.1, 17.8)
- added TP69: TestPoint, TestPoint:TestPoint_Pad_D1.0mm, F.Cu at (175.0, 62.3)
- added TP7: TestPoint, TestPoint:TestPoint_Pad_D1.0mm, F.Cu at (177.0, 48.6)
- added TP70: TestPoint, TestPoint:TestPoint_Pad_D1.0mm, F.Cu at (172.0, 65.3)
- added TP71: TestPoint, TestPoint:TestPoint_Pad_D1.0mm, F.Cu at (200.7, 37.3)
- added TP72: TestPoint, TestPoint:TestPoint_Pad_D1.0mm, F.Cu at (209.5, 30.0)
- added TP73: TestPoint, TestPoint:TestPoint_Pad_D1.0mm, F.Cu at (197.3, 40.4)
- added TP74: TestPoint, TestPoint:TestPoint_Pad_D1.0mm, F.Cu at (209.5, 26.9)
- added TP75: TestPoint, TestPoint:TestPoint_Pad_D1.0mm, F.Cu at (194.2, 42.0)
- added TP76: TestPoint, TestPoint:TestPoint_Pad_D1.0mm, F.Cu at (189.2, 48.1)
- added TP77: TestPoint, TestPoint:TestPoint_Pad_D1.0mm, F.Cu at (214.5, 23.9)
- added TP79: TestPoint, TestPoint:TestPoint_Pad_D1.0mm, F.Cu at (181.1, 58.6)
- added TP8: TestPoint, TestPoint:TestPoint_Pad_D1.0mm, F.Cu at (161.8, 64.1)
- added TP80: TestPoint, TestPoint:TestPoint_Pad_D1.0mm, F.Cu at (212.6, 26.9)
- added TP81: TestPoint, TestPoint:TestPoint_Pad_D1.0mm, F.Cu at (203.8, 32.1)
- added TP82: TestPoint, TestPoint:TestPoint_Pad_D1.0mm, F.Cu at (178.1, 61.7)
- added TP83: TestPoint, TestPoint:TestPoint_Pad_D1.0mm, F.Cu at (175.0, 65.3)
- added TP84: TestPoint, TestPoint:TestPoint_Pad_D1.0mm, F.Cu at (200.3, 40.4)
- added TP85: TestPoint, TestPoint:TestPoint_Pad_D1.0mm, F.Cu at (192.3, 48.1)
- added TP86: TestPoint, TestPoint:TestPoint_Pad_D1.0mm, F.Cu at (197.3, 43.4)
- added TP87: TestPoint, TestPoint:TestPoint_Pad_D1.0mm, F.Cu at (190.0, 51.2)
- added TP88: TestPoint, TestPoint:TestPoint_Pad_D1.0mm, F.Cu at (217.6, 23.9)
- added TP89: TestPoint, TestPoint:TestPoint_Pad_D1.0mm, F.Cu at (209.9, 33.0)
- added TP9: TestPoint, TestPoint:TestPoint_Pad_D1.0mm, F.Cu at (201.4, 25.1)
- added TP90: TestPoint, TestPoint:TestPoint_Pad_D1.0mm, F.Cu at (181.1, 61.7)
- added TP91: TestPoint, TestPoint:TestPoint_Pad_D1.0mm, F.Cu at (184.2, 55.6)
- added TP92: TestPoint, TestPoint:TestPoint_Pad_D1.0mm, F.Cu at (203.8, 38.2)
- added TP93: TestPoint, TestPoint:TestPoint_Pad_D1.0mm, F.Cu at (212.6, 30.0)
- added TP94: TestPoint, TestPoint:TestPoint_Pad_D1.0mm, F.Cu at (215.6, 26.9)
- added TP95: TestPoint, TestPoint:TestPoint_Pad_D1.0mm, F.Cu at (184.2, 58.6)
- added TP96: TestPoint, TestPoint:TestPoint_Pad_D1.0mm, F.Cu at (187.2, 54.2)
- added TP98: TestPoint, TestPoint:TestPoint_Pad_D1.0mm, F.Cu at (216.0, 33.0)
- added TP99: TestPoint, TestPoint:TestPoint_Pad_D1.0mm, F.Cu at (187.2, 57.3)
- D112, D114: value ledred -> SS210; footprint LED_SMD:LED_0603_1608Metric -> Diode_SMD:D_SMA
- J22: renamed from D84; value ledred -> USB_B_Micro; footprint LED_SMD:LED_0603_1608Metric -> Connector_USB:USB_Micro-B_Molex-105017-0001
- J27: value USB_B_Micro -> Conn_01x07_Male; footprint Connector_USB:USB_Micro-B_Molex-105017-0001 -> Connector_PinHeader_2.54mm:PinHeader_1x07_P2.54mm_Vertical
- J3: renamed from D43; value ledred -> USB_B_Micro; footprint LED_SMD:LED_0603_1608Metric -> Connector_USB:USB_Micro-B_Molex-105017-0001
- TP116: renamed from D143; value ledred -> TestPoint; footprint LED_SMD:LED_0603_1608Metric -> TestPoint:TestPoint_Pad_D1.0mm
- TP128: renamed from J1; value USB_B_Micro -> TestPoint; footprint Connector_USB:USB_Micro-B_Molex-105017-0001 -> TestPoint:TestPoint_Pad_D1.0mm
- TP18: renamed from D102; value ledred -> TestPoint; footprint LED_SMD:LED_0603_1608Metric -> TestPoint:TestPoint_Pad_D1.0mm
- TP40: renamed from D111; value ledred -> TestPoint; footprint LED_SMD:LED_0603_1608Metric -> TestPoint:TestPoint_Pad_D1.0mm
- TP59: renamed from D119; value ledred -> TestPoint; footprint LED_SMD:LED_0603_1608Metric -> TestPoint:TestPoint_Pad_D1.0mm
- TP78: renamed from D127; value ledred -> TestPoint; footprint LED_SMD:LED_0603_1608Metric -> TestPoint:TestPoint_Pad_D1.0mm
- TP97: renamed from D135; value ledred -> TestPoint; footprint LED_SMD:LED_0603_1608Metric -> TestPoint:TestPoint_Pad_D1.0mm
- moved D28 240.0 mm to (59.8, 139.9), turned to 180 degrees
- moved D24 226.5 mm to (59.8, 134.5), turned to 180 degrees
- moved D39 208.4 mm to (59.8, 136.3), turned to 180 degrees
- moved TP40 196.3 mm to (55.4, 140.2)
- moved D49 187.3 mm to (194.3, 14.5), turned to 0 degrees
- moved J3 182.2 mm to (51.8, 83.7), turned to 270 degrees
- moved D32 177.1 mm to (59.8, 138.1), turned to 180 degrees
- moved D40 176.7 mm to (59.8, 141.8), turned to 180 degrees
- moved D61 176.1 mm to (189.7, 22.3), turned to 0 degrees
- moved D63 148.1 mm to (172.4, 39.2), turned to 0 degrees
- moved D19 142.2 mm to (128.4, 28.8)
- moved D50 140.7 mm to (161.4, 45.7), turned to 0 degrees
- moved TP128 140.7 mm to (193.3, 57.3), turned to 0 degrees
- moved D26 139.8 mm to (128.4, 31.4)
- moved D62 139.7 mm to (165.4, 47.7), turned to 0 degrees
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- renumbered C5 to C6, C6 to C7, C7 to C8, D109 to D113, J24 to J23, J20 to J24, J19 to J25
Connections:
- C7 pad 1: Net-(C6-Pad1) (its old number) -> Net-(C7-Pad1)
- D112 pad 1: GND -> VIN
- D113 pad 1: Net-(C6-Pad1) (its old number) -> VIN
- D113 pad 2: Net-(D109-Pad2) -> Net-(D113-Pad2)
- D114 pad 1: GND -> VIN
- F1 pad 1: Net-(D109-Pad2) -> Net-(C7-Pad1)
- J10 pad 1: Net-(D52-Pad2) -> Net-(D42-Pad2)
- J10 pad 2: Net-(D53-Pad2) -> Net-(D55-Pad2)
- J10 pad 3: Net-(D64-Pad2) -> Net-(D50-Pad2)
- J10 pad 4: Net-(D65-Pad2) -> Net-(J10-Pad4)
- J10 pad 5: Net-(D54-Pad2) -> Net-(D46-Pad2)
- J10 pad 6: Net-(D66-Pad2) -> Net-(D56-Pad2)
- J11 pad 1: Net-(D55-Pad2) -> Net-(D43-Pad2)
- J11 pad 2: Net-(D56-Pad2) -> Net-(D57-Pad2)
- J11 pad 3: Net-(D67-Pad2) -> Net-(D51-Pad2)
- J11 pad 4: Net-(D68-Pad2) -> Net-(J11-Pad4)
- J11 pad 5: Net-(D57-Pad2) -> Net-(D47-Pad2)
- J11 pad 6: Net-(D69-Pad2) -> Net-(D58-Pad2)
- J12 pad 1: Net-(D58-Pad2) -> Net-(D44-Pad2)
- J12 pad 3: Net-(D70-Pad2) -> Net-(D52-Pad2)
- J12 pad 4: Net-(D71-Pad2) -> Net-(J12-Pad4)
- J12 pad 5: Net-(D60-Pad2) -> Net-(D48-Pad2)
- J12 pad 6: Net-(D72-Pad2) -> Net-(D60-Pad2)
- J13 pad 1: Net-(D73-Pad2) -> Net-(D61-Pad2)
- J13 pad 2: Net-(D74-Pad2) -> Net-(D73-Pad2)
- J13 pad 3: Net-(D82-Pad2) -> Net-(D69-Pad2)
- J13 pad 4: Net-(D83-Pad2) -> Net-(J13-Pad4)
- J13 pad 5: Net-(D75-Pad2) -> Net-(D65-Pad2)
- J13 pad 6: Net-(D84-Pad2) -> Net-(D74-Pad2)
- J14 pad 1: Net-(D76-Pad2) -> Net-(D62-Pad2)
- J14 pad 2: Net-(D77-Pad2) -> Net-(D75-Pad2)
- J14 pad 3: Net-(D85-Pad2) -> Net-(D70-Pad2)
- J14 pad 4: Net-(D86-Pad2) -> Net-(J14-Pad4)
- J14 pad 5: Net-(D78-Pad2) -> Net-(D66-Pad2)
- J14 pad 6: Net-(D87-Pad2) -> Net-(D76-Pad2)
- J15 pad 1: Net-(D79-Pad2) -> Net-(D63-Pad2)
- J15 pad 2: Net-(D80-Pad2) -> Net-(D77-Pad2)
- J15 pad 3: Net-(D88-Pad2) -> Net-(D71-Pad2)
- J15 pad 4: Net-(D89-Pad2) -> Net-(J15-Pad4)
- J15 pad 5: Net-(D81-Pad2) -> Net-(D67-Pad2)
- J15 pad 6: Net-(D90-Pad2) -> Net-(D78-Pad2)
- J16 pad 1: Net-(D91-Pad2) -> Net-(D64-Pad2)
- J16 pad 2: Net-(D92-Pad2) -> Net-(D79-Pad2)
- J16 pad 3: Net-(D100-Pad2) -> Net-(D72-Pad2)
- J16 pad 4: Net-(D101-Pad2) -> Net-(J16-Pad4)
- J16 pad 5: Net-(D93-Pad2) -> Net-(D68-Pad2)
- J16 pad 6: Net-(D102-Pad2) -> Net-(D80-Pad2)
- J17 pad 1: Net-(D94-Pad2) -> Net-(D81-Pad2)
- J17 pad 2: Net-(D95-Pad2) -> Net-(D93-Pad2)
- J17 pad 3: Net-(D103-Pad2) -> Net-(D89-Pad2)
- J17 pad 4: Net-(D104-Pad2) -> Net-(J17-Pad4)
- J17 pad 5: Net-(D96-Pad2) -> Net-(D85-Pad2)
- J17 pad 6: Net-(D105-Pad2) -> Net-(D94-Pad2)
- J18 pad 1: Net-(D97-Pad2) -> Net-(D82-Pad2)
- J18 pad 2: Net-(D98-Pad2) -> Net-(D95-Pad2)
- J18 pad 3: Net-(D106-Pad2) -> Net-(D90-Pad2)
- J18 pad 4: Net-(D107-Pad2) -> Net-(J18-Pad4)
- J18 pad 5: Net-(D99-Pad2) -> Net-(D86-Pad2)
- J18 pad 6: Net-(D108-Pad2) -> Net-(D96-Pad2)
- J2 pad 1: Net-(D4-Pad2) -> Net-(D2-Pad2)
- J2 pad 2: Net-(D5-Pad2) -> Net-(D15-Pad2)
- J2 pad 3: Net-(D16-Pad2) -> Net-(D10-Pad2)
- J2 pad 4: Net-(D17-Pad2) -> Net-(J2-Pad4)
- J2 pad 6: Net-(D18-Pad2) -> Net-(D16-Pad2)
- J21 pad 1: Net-(D110-Pad2) -> Net-(D101-Pad2)
- J21 pad 2: Net-(D111-Pad2) -> Net-(D107-Pad2)
- J21 pad 3: Net-(D119-Pad2) -> Net-(D105-Pad2)
- J21 pad 5: Net-(D112-Pad2) -> Net-(D103-Pad2)
- J21 pad 6: Net-(D121-Pad2) -> Net-(D108-Pad2)
- J22 pad 1: GND -> Net-(D102-Pad2)
- J22 pad 2: Net-(D84-Pad2) -> Net-(D109-Pad2)
- J23 pad 1: TEST_VBUS -> TEST1
- J23 pad 2: TEST_DP -> TEST2
- J23 pad 3: TEST_DM -> TEST3
- J23 pad 4: TEST_GND -> TEST5
- J23 pad 5: TEST_SHIELD -> TEST6
- J24 pad 1: Net-(F1-Pad2) -> Net-(D112-Pad2)
- J25 pad 1: Net-(F1-Pad2) -> Net-(D113-Pad2)
- J26 pad 1: Net-(D131-Pad2) -> Net-(D114-Pad2)
- J26 pad 2: Net-(D132-Pad2) -> (no net)
- J26 pad 3: Net-(D140-Pad2) -> (no net)
- J26 pad 4: Net-(D141-Pad2) -> (no net)
- J26 pad 5: Net-(D133-Pad2) -> GND
- J27 pad 1: Net-(D134-Pad2) -> TEST1
- J27 pad 2: Net-(D135-Pad2) -> TEST2
- J27 pad 3: Net-(D143-Pad2) -> TEST3
- J27 pad 4: Net-(D144-Pad2) -> TEST4
- J27 pad 5: Net-(D136-Pad2) -> TEST5
- J27 pad 6: Net-(D145-Pad2) -> TEST6
- J3 pad 1: GND -> Net-(D3-Pad2)
- J3 pad 2: Net-(D43-Pad2) -> Net-(D17-Pad2)
- J4 pad 1: Net-(D10-Pad2) -> Net-(D4-Pad2)
- J4 pad 2: Net-(D11-Pad2) -> Net-(D19-Pad2)
- J4 pad 3: Net-(D22-Pad2) -> Net-(D12-Pad2)
- J4 pad 4: Net-(D23-Pad2) -> Net-(J4-Pad4)
- J4 pad 5: Net-(D12-Pad2) -> Net-(D8-Pad2)
- J4 pad 6: Net-(D24-Pad2) -> Net-(D20-Pad2)
- J5 pad 1: Net-(D25-Pad2) -> Net-(D21-Pad2)
- J5 pad 2: Net-(D26-Pad2) -> Net-(D33-Pad2)
- J5 pad 3: Net-(D37-Pad2) -> Net-(D29-Pad2)
- J5 pad 4: Net-(D38-Pad2) -> Net-(J5-Pad4)
- J5 pad 5: Net-(D27-Pad2) -> Net-(D25-Pad2)
- J5 pad 6: Net-(D39-Pad2) -> Net-(D34-Pad2)
- J6 pad 1: Net-(D28-Pad2) -> Net-(D22-Pad2)
- J6 pad 2: Net-(D29-Pad2) -> Net-(D35-Pad2)
- J6 pad 3: Net-(D40-Pad2) -> Net-(D30-Pad2)
- J6 pad 4: Net-(D41-Pad2) -> Net-(J6-Pad4)
- J6 pad 5: Net-(D30-Pad2) -> Net-(D26-Pad2)
- J6 pad 6: Net-(D42-Pad2) -> Net-(D36-Pad2)
- J7 pad 1: Net-(D31-Pad2) -> Net-(D23-Pad2)
- J7 pad 2: Net-(D32-Pad2) -> Net-(D37-Pad2)
- J7 pad 3: Net-(D43-Pad2) -> Net-(D31-Pad2)
- J7 pad 4: Net-(D44-Pad2) -> Net-(J7-Pad4)
- J7 pad 5: Net-(D33-Pad2) -> Net-(D27-Pad2)
- J7 pad 6: Net-(D45-Pad2) -> Net-(D38-Pad2)
- J8 pad 1: Net-(D34-Pad2) -> Net-(D24-Pad2)
- J8 pad 2: Net-(D35-Pad2) -> Net-(D39-Pad2)
- J8 pad 3: Net-(D46-Pad2) -> Net-(D32-Pad2)
- J8 pad 4: Net-(D47-Pad2) -> Net-(J8-Pad4)
- J8 pad 5: Net-(D36-Pad2) -> Net-(D28-Pad2)
- J8 pad 6: Net-(D48-Pad2) -> Net-(D40-Pad2)
- J9 pad 1: Net-(D49-Pad2) -> Net-(D41-Pad2)
- J9 pad 2: Net-(D50-Pad2) -> Net-(D53-Pad2)
- J9 pad 3: Net-(D61-Pad2) -> Net-(D49-Pad2)
- J9 pad 4: Net-(D62-Pad2) -> Net-(J9-Pad4)
- J9 pad 5: Net-(D51-Pad2) -> Net-(D45-Pad2)
- J9 pad 6: Net-(D63-Pad2) -> Net-(D54-Pad2)
- TP116 pad 1: GND -> Net-(D92-Pad2)
- TP128 pad 1: Net-(D1-Pad2) -> Net-(D104-Pad2)
- TP18 pad 1: GND -> Net-(D10-Pad2)
- TP40 pad 1: GND -> Net-(D28-Pad2)
- TP59 pad 1: GND -> Net-(D44-Pad2)
- TP78 pad 1: GND -> Net-(J13-Pad4)
- TP97 pad 1: GND -> Net-(D94-Pad2)
- U2 pad 10: TEST_GND -> Net-(R7-Pad1)
- U2 pad 11: TEST_SHIELD -> Net-(R8-Pad1)
- U2 pad 12: (no net) -> LAST
- U2 pad 3: TEST_VBUS -> Net-(R3-Pad1)
- U2 pad 4: TEST_DP -> Net-(R4-Pad1)
- U2 pad 5: TEST_DM -> Net-(R5-Pad1)
- U3 pad 10: TEST_GND -> Net-(R7-Pad1)
- U3 pad 11: TEST_SHIELD -> Net-(R8-Pad1)
- U3 pad 12: GND -> LAST
- U3 pad 2: TEST_VBUS -> Net-(R3-Pad1)
- U3 pad 3: TEST_DP -> Net-(R4-Pad1)
- U3 pad 4: TEST_DM -> Net-(R5-Pad1)
- U5 pad 3: Net-(C6-Pad1) (its old number) -> Net-(C7-Pad1)
Routing:
- net Net-(D40-Pad2): track 0.00 -> 19.1 mm
- net GND: track 0.00 -> 7.26 mm
- net Net-(D24-Pad2): track 0.00 -> 7.21 mm
- net Net-(D32-Pad2): track 0.00 -> 6.57 mm
- net Net-(D39-Pad2): track 0.00 -> 6.39 mm
- net Net-(D28-Pad2): track 0.00 -> 6.13 mm
- net Net-(J8-Pad4): track 0.00 -> 3.78 mm

Commit message: routing
Parts:
- U4: value 74HC04 -> 74AHC1G04; footprint Package_SO:SOIC-14_3.9x8.7mm_P1.27mm -> Package_TO_SOT_SMD:SOT-353_SC-70-5
- moved C1 196.7 mm to (97.6, 83.0)
- moved C6 193.7 mm to (99.8, 81.5), turned to 270 degrees
- moved R2 192.9 mm to (99.8, 79.3), turned to 270 degrees
- moved TP61 190.5 mm to (73.0, 143.7)
- moved TP39 189.9 mm to (56.1, 129.3)
- moved TP32 187.4 mm to (59.0, 117.0)
- moved TP53 187.1 mm to (67.6, 143.5)
- moved R1 182.7 mm to (97.5, 78.1)
- moved C7 182.7 mm to (109.1, 65.6)
- moved D27 179.2 mm to (62.4, 129.1), turned to 180 degrees
- moved TP31 178.5 mm to (56.1, 113.0)
- moved TP34 177.6 mm to (59.0, 127.9)
- moved TP30 177.6 mm to (59.0, 106.1)
- moved TP43 176.7 mm to (56.1, 126.6)
- moved D49 174.9 mm to (71.0, 138.5), turned to 270 degrees
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Connections:
- D111 pad 2: Net-(D111-Pad2) -> SYNC
- R3 pad 2: TEST1 -> SYNC
- R4 pad 2: TEST2 -> TEST1
- R5 pad 2: TEST3 -> TEST2
- R6 pad 2: TEST5 -> TEST3
- R7 pad 2: TEST6 -> TEST5
- R8 pad 2: TEST4 -> TEST6
- R9 pad 1: LAST -> Net-(R9-Pad1)
- R9 pad 2: Net-(D111-Pad2) -> TEST4
- U2 pad 12: LAST -> Net-(R9-Pad1)
- U3 pad 10: Net-(R7-Pad1) -> Net-(U3-Pad1)
- U3 pad 11: Net-(R8-Pad1) -> Net-(R4-Pad1)
- U3 pad 12: LAST -> Net-(R3-Pad1)
- U3 pad 14: (no net) -> +3V3
- U3 pad 2: Net-(R3-Pad1) -> Net-(R9-Pad1)
- U3 pad 3: Net-(R4-Pad1) -> Net-(R8-Pad1)
- U3 pad 4: Net-(R5-Pad1) -> Net-(R7-Pad1)
- U3 pad 7: (no net) -> GND
- U3 pad 9: Net-(U3-Pad1) -> Net-(R5-Pad1)
- U4 pad 1: Net-(U3-Pad13) -> (no net)
- U4 pad 2: Net-(U2-Pad1) -> Net-(U3-Pad13)
- U4 pad 3: (no net) -> GND
- U4 pad 4: (no net) -> Net-(U2-Pad1)
- U4 pad 5: (no net) -> +3V3
Routing:
- net TEST6: track 0.00 -> 48.0 mm
- net Net-(R4-Pad1): track 0.00 -> 36.4 mm
- net Net-(R5-Pad1): track 0.00 -> 32.9 mm
- net TEST5: track 0.00 -> 32.3 mm
- net Net-(U1-Pad3): track 0.00 -> 31.3 mm
- net TEST3: track 0.00 -> 31.3 mm
- net TEST2: track 0.00 -> 31.0 mm
- net TEST1: track 0.00 -> 31.0 mm
- net Net-(R3-Pad1): track 0.00 -> 25.4 mm
- net Net-(R8-Pad1): track 0.00 -> 25.4 mm, vias 0 -> 2
- net Net-(R9-Pad1): track 0.00 -> 23.6 mm
- net Net-(R7-Pad1): track 0.00 -> 22.7 mm
- net Net-(D14-Pad2): track 0.00 -> 21.9 mm
- net Net-(R6-Pad1): track 0.00 -> 21.7 mm, vias 0 -> 2
- net Net-(D40-Pad2): track 19.1 -> 0.00 mm
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- added copper zone on In2.Cu, net +3V3
- added copper zone on In1.Cu, net GND
Other:
- copper layers 2 -> 4

Commit message: routing
Parts:
- moved D104 167.5 mm to (135.3, 60.3)
- moved D103 164.2 mm to (132.7, 73.0)
- moved TP130 151.8 mm to (142.9, 62.2)
- moved D102 149.7 mm to (135.9, 66.0)
- moved TP128 146.6 mm to (142.9, 60.3)
- moved D107 146.3 mm to (132.7, 76.8)
- moved TP121 145.2 mm to (139.7, 71.1)
- moved TP107 141.2 mm to (143.5, 88.9)
- moved D91 139.7 mm to (138.4, 96.5)
- moved TP127 138.9 mm to (142.9, 72.4)
- moved TP132 136.9 mm to (139.7, 63.5)
- moved TP100 136.3 mm to (140.3, 81.9)
- moved TP126 135.6 mm to (139.7, 61.6)
- moved TP124 130.3 mm to (139.7, 74.3)
- moved TP112 129.7 mm to (142.9, 83.2)
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
Commit message: routing
Parts:
- moved C2 159.6 mm to (90.8, 87.6)
- moved D84 134.7 mm to (136.7, 87.3)
- moved D92 130.2 mm to (136.7, 83.7)
- moved D100 125.8 mm to (136.7, 80.1)
- moved D99 98.9 mm to (136.7, 85.5)
- moved D88 88.2 mm to (136.7, 81.9)
- moved D107 4.56 mm to (136.7, 74.6)
- moved D103 4.47 mm to (136.7, 71.0)
- moved J19 4.18 mm to (147.3, 94.6)
- moved TP105 4.06 mm to (143.0, 98.0)
- moved TP111 3.96 mm to (143.0, 92.5)
- moved D98 3.84 mm to (136.7, 91.0)
- moved TP115 3.74 mm to (143.0, 95.3)
- moved TP99 3.74 mm to (140.1, 91.2)
- moved TP119 3.60 mm to (140.1, 96.6)
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
Commit message: routing
Parts:
- moved TP84 1.08 mm to (140.1, 126.6)
- moved TP92 0.99 mm to (143.0, 127.9)
- moved TP96 0.90 mm to (140.1, 129.3)
- moved TP88 0.53 mm to (143.0, 125.2)
Routing:
- net Net-(D34-Pad2): track 0.00 -> 21.9 mm
- net Net-(D56-Pad2): track 0.00 -> 21.7 mm
- net Net-(D54-Pad2): track 0.00 -> 21.7 mm
- net Net-(D60-Pad2): track 0.00 -> 21.7 mm
- net Net-(D74-Pad2): track 0.00 -> 21.7 mm
- net Net-(D58-Pad2): track 0.00 -> 21.7 mm
- net Net-(D36-Pad2): track 0.00 -> 21.7 mm
- net Net-(D20-Pad2): track 0.00 -> 21.7 mm
- net Net-(D16-Pad2): track 0.00 -> 21.7 mm
- net Net-(D78-Pad2): track 0.00 -> 21.3 mm
- net Net-(D110-Pad2): track 0.00 -> 21.3 mm
- net Net-(D80-Pad2): track 0.00 -> 21.2 mm
- net Net-(D100-Pad2): track 0.00 -> 21.2 mm
- net Net-(D76-Pad2): track 0.00 -> 21.1 mm
- net Net-(D40-Pad2): track 0.00 -> 21.1 mm
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
Commit message: lib
Parts:
- H1, H2, H3, H4: value MountingHole -> MountingHole_Pad; footprint MountingHole:MountingHole_3.5mm -> MountingHole:MountingHole_3.2mm_M3_Pad
- moved H2 92.8 mm to (146.6, 53.4)
- moved H4 92.8 mm to (146.5, 146.6)
- moved H1 0.47 mm to (53.4, 53.4)
- moved H3 0.43 mm to (53.4, 146.6)
Connections:
- H1 pad 1: (no net) -> GND
- H2 pad 1: (no net) -> GND
- H3 pad 1: (no net) -> GND
- H4 pad 1: (no net) -> GND

Commit message: id
Parts:
- added D115: ledred, LED_SMD:LED_0603_1608Metric, F.Cu at (133.8, 74.6)
- added R10: 10k, Resistor_SMD:R_0402_1005Metric, F.Cu at (133.8, 72.3)
- moved TP124 6.55 mm to (133.8, 70.5)
Routing:
- net Net-(J21-Pad4): track 5.77 -> 17.3 mm, vias 0 -> 2
- net Net-(D115-Pad1): track 0.00 -> 1.74 mm
- net +3V3: track 11.9 -> 13.3 mm, vias 5 -> 6
Changed lines of the file:
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@@
     (thickness 1.6)
     (drawings 4)
-    (tracks 945)
+    (tracks 957)
     (zones 0)
-    (modules 301)
-    (nets 163)
+    (modules 303)
+    (nets 164)
   )
   (page A4)
@@
   )
   (setup
-    (last_trace_width 0.25)
+    (last_trace_width 0.4)
     (user_trace_width 0.4)
     (user_trace_width 0.5)
@@
   (net 161 SYNC)
   (net 162 "Net-(R9-Pad1)")
+  (net 163 "Net-(D115-Pad1)")
   (net_class Default "This is the default net class."
     (clearance 0.2)
@@
     (add_net "Net-(D113-Pad2)")
     (add_net "Net-(D114-Pad2)")
+    (add_net "Net-(D115-Pad1)")
     (add_net "Net-(D12-Pad2)")
     (add_net "Net-(D13-Pad2)")
@@
   )
   (module TestPoint:TestPoint_Pad_D1.0mm (layer F.Cu)
-    (at 140.1 72.130914)
+    (at 133.7564 70.500913)
     (descr "SMD pad as test Point, diameter 1.0mm")
     (tags "test point SMD pad")
@@
       (net 2 GND))
   )
+  (module LED_SMD:LED_0603_1608Metric (layer F.Cu)
+    (at 133.7564 74.640913 270)
+    (descr "LED SMD 0603 (1608 Metric), square (rectangular) end terminal, IPC_7351 nominal, (Body size source: http://www.tortai-tech.com/upload/download/2011102023233369053.pdf), generated with kicad-footprint-generator")
+    (tags diode)
+    (attr smd)
+    (fp_text reference D115 (at 0 -1.43 90) (layer F.SilkS) hide
+      (effects (font (size 1 1) (thickness 0.15)))
+    )
+    (fp_text value ledred (at 0 1.43 90) (layer F.Fab)
+      (effects (font (size 1 1) (thickness 0.15)))
+    )
+    (fp_line (start 0.8 -0.4) (end -0.5 -0.4) (layer F.Fab) (width 0.1))
+    (fp_line (start -0.5 -0.4) (end -0.8 -0.1) (layer F.Fab) (width 0.1))
+    (fp_line (start -0.8 -0.1) (end -0.8 0.4) (layer F.Fab) (width 0.1))
+    (fp_line (start -0.8 0.4) (end 0.8 0.4) (layer F.Fab) (width 0.1))
+    (fp_line (start 0.8 0.4) (end 0.8 -0.4) (layer F.Fab) (width 0.1))
+    (fp_line (start 0.8 -0.735) (end -1.485 -0.735) (layer F.SilkS) (width 0.12))
+    (fp_line (start -1.485 -0.735) (end -1.485 0.735) (layer F.SilkS) (width 0.12))
+    (fp_line (start -1.485 0.735) (end 0.8 0.735) (layer F.SilkS) (width 0.12))
+    (fp_line (start -1.48 0.73) (end -1.48 -0.73) (layer F.CrtYd) (width 0.05))
+    (fp_line (start -1.48 -0.73) (end 1.48 -0.73) (layer F.CrtYd) (width 0.05))
+    (fp_line (start 1.48 -0.73) (end 1.48 0.73) (layer F.CrtYd) (width 0.05))
+    (fp_line (start 1.48 0.73) (end -1.48 0.73) (layer F.CrtYd) (width 0.05))
+    (fp_text user %R (at 0 0 90) (layer F.Fab)
+      (effects (font (size 0.4 0.4) (thickness 0.06)))
+    )
+    (pad 1 smd roundrect (at -0.7875 0 270) (size 0.875 0.95) (layers F.Cu F.Paste F.Mask) (roundrect_rratio 0.25)
+      (net 163 "Net-(D115-Pad1)"))
+    (pad 2 smd roundrect (at 0.7875 0 270) (size 0.875 0.95) (layers F.Cu F.Paste F.Mask) (roundrect_rratio 0.25)
+      (net 3 +3V3))
+    (model ${KISYS3DMOD}/LED_SMD.3dshapes/LED_0603_1608Metric.wrl
+      (at (xyz 0 0 0))
+      (scale (xyz 1 1 1))
+      (rotate (xyz 0 0 0))
+    )
+  )
+  (module Resistor_SMD:R_0402_1005Metric (layer F.Cu)
+    (at 133.7564 72.310913)
+    (descr "Resistor SMD 0402 (1005 Metric), square (rectangular) end terminal, IPC_7351 nominal, (Body size source: http://www.tortai-tech.com/upload/download/2011102023233369053.pdf), generated with kicad-footprint-generator")
+    (tags resistor)
+    (attr smd)
+    (fp_text reference R10 (at 0 -1.17) (layer F.SilkS) hide
+      (effects (font (size 1 1) (thickness 0.15)))
+    )
+    (fp_text value 10k (at 0 1.17) (layer F.Fab)
+      (effects (font (size 1 1) (thickness 0.15)))
+    )
+    (fp_line (start -0.5 0.25) (end -0.5 -0.25) (layer F.Fab) (width 0.1))
+    (fp_line (start -0.5 -0.25) (end 0.5 -0.25) (layer F.Fab) (width 0.1))
+    (fp_line (start 0.5 -0.25) (end 0.5 0.25) (layer F.Fab) (width 0.1))
+    (fp_line (start 0.5 0.25) (end -0.5 0.25) (layer F.Fab) (width 0.1))
+    (fp_line (start -0.93 0.47) (end -0.93 -0.47) (layer F.CrtYd) (width 0.05))
+    (fp_line (start -0.93 -0.47) (end 0.93 -0.47) (layer F.CrtYd) (width 0.05))
+    (fp_line (start 0.93 -0.47) (end 0.93 0.47) (layer F.CrtYd) (width 0.05))
+    (fp_line (start 0.93 0.47) (end -0.93 0.47) (layer F.CrtYd) (width 0.05))
+    (fp_text user %R (at 0 0) (layer F.Fab)
+      (effects (font (size 0.25 0.25) (thickness 0.04)))
+    )
+    (pad 1 smd roundrect (at -0.485 0) (size 0.59 0.64) (layers F.Cu F.Paste F.Mask) (roundrect_rratio 0.25)
+      (net 163 "Net-(D115-Pad1)"))
+    (pad 2 smd roundrect (at 0.485 0) (size 0.59 0.64) (layers F.Cu F.Paste F.Mask) (roundrect_rratio 0.25)
+      (net 146 "Net-(J21-Pad4)"))
+    (model ${KISYS3DMOD}/Resistor_SMD.3dshapes/R_0402_1005Metric.wrl
+      (at (xyz 0 0 0))
+      (scale (xyz 1 1 1))
+      (rotate (xyz 0 0 0))
+    )
+  )
   (gr_line (start 50 50) (end 50 150) (layer Edge.Cuts) (width 0.05))
   (gr_line (start 150 50) (end 150 150) (layer Edge.Cuts) (width 0.05))
@@
   (via (at 124.968 102.108) (size 0.8) (drill 0.4) (layers F.Cu B.Cu) (net 3))
   (segment (start 124.968 101.069) (end 124.968 102.108) (width 0.25) (layer F.Cu) (net 3) (status 10))
+  (via (at 133.7564 76.835914) (size 0.8) (drill 0.4) (layers F.Cu B.Cu) (net 3))
+  (segment (start 133.7564 75.428413) (end 133.7564 76.835914) (width 0.4) (layer F.Cu) (net 3))
   (segment (start 56.9832 58.7455) (end 56.9832 58.5252) (width 0.25) (layer F.Cu) (net 5) (status 30))
   (segment (start 55.1035 60.6252) (end 56.9832 58.7455) (width 0.25) (layer F.Cu) (net 5) (status 20))
@@
   (segment (start 140.13 83.046628) (end 140.1 83.016628) (width 0.4) (layer F.Cu) (net 145) (status 30))
   (segment (start 145.8575 83.046628) (end 140.13 83.046628) (width 0.4) (layer F.Cu) (net 145) (status 30))
-  (segment (start 140.13 72.160914) (end 140.1 72.130914) (width 0.4) (layer F.Cu) (net 146) (status 30))
-  (segment (start 145.8575 72.160914) (end 140.13 72.160914) (width 0.4) (layer F.Cu) (net 146) (status 30))
+  (via (at 140.4366 72.2122) (size 0.8) (drill 0.4) (layers F.Cu B.Cu) (net 146))
+  (segment (start 140.487886 72.160914) (end 140.4366 72.2122) (width 0.4) (layer F.Cu) (net 146))
+  (segment (start 145.8575 72.160914) (end 140.487886 72.160914) (width 0.4) (layer F.Cu) (net 146))
+  (segment (start 140.4366 72.2122) (end 137.4648 69.2404) (width 0.4) (layer B.Cu) (net 146))
+  (via (at 133.7564 68.785913) (size 0.8) (drill 0.4) (layers F.Cu B.Cu) (net 146))
+  (segment (start 134.210887 69.2404) (end 133.7564 68.785913) (width 0.4) (layer B.Cu) (net 146))
+  (segment (start 137.4648 69.2404) (end 134.210887 69.2404) (width 0.4) (layer B.Cu) (net 146))
+  (segment (start 133.7564 68.785913) (end 133.7564 70.500913) (width 0.4) (layer F.Cu) (net 146))
+  (segment (start 134.2414 70.985913) (end 134.2414 72.310913) (width 0.4) (layer F.Cu) (net 146))
+  (segment (start 133.7564 70.500913) (end 134.2414 70.985913) (width 0.4) (layer F.Cu) (net 146))
   (segment (start 140.13 61.2752) (end 140.1 61.2452) (width 0.4) (layer F.Cu) (net 147) (status 30))
   (segment (start 145.8971 61.2752) (end 140.13 61.2752) (width 0.4) (layer F.Cu) (net 147) (status 30))
@@
   (segment (start 118.872 98.552) (end 120.04699 99.72699) (width 0.25) (layer F.Cu) (net 162))
   (segment (start 116.020599 94.759251) (end 116.31659 95.055242) (width 0.25) (layer F.Cu) (net 162))
+  (segment (start 133.2714 73.368413) (end 133.7564 73.853413) (width 0.4) (layer F.Cu) (net 163))
+  (segment (start 133.2714 72.310913) (end 133.2714 73.368413) (width 0.4) (layer F.Cu) (net 163))
   (zone (net 2) (net_name GND) (layer In1.Cu) (hatch edge 0.508)
     (connect_pads (clearance 0.508))

Commit message: id
Parts:
- added D116: ledred, LED_SMD:LED_0603_1608Metric, F.Cu at (133.8, 118.2)
- added D117: ledred, LED_SMD:LED_0603_1608Metric, F.Cu at (133.8, 107.5)
- added D118: ledred, LED_SMD:LED_0603_1608Metric, F.Cu at (133.8, 96.4)
- added D119: ledred, LED_SMD:LED_0603_1608Metric, F.Cu at (133.8, 85.5)
- added D120: ledred, LED_SMD:LED_0603_1608Metric, F.Cu at (133.7, 63.8)
- added R11: 10k, Resistor_SMD:R_0402_1005Metric, F.Cu at (133.8, 115.9)
- added R12: 10k, Resistor_SMD:R_0402_1005Metric, F.Cu at (133.8, 105.1)
- added R13: 10k, Resistor_SMD:R_0402_1005Metric, F.Cu at (133.8, 94.1)
- added R14: 10k, Resistor_SMD:R_0402_1005Metric, F.Cu at (133.8, 83.2)
- added R15: 10k, Resistor_SMD:R_0402_1005Metric, F.Cu at (133.8, 61.4)
- moved TP102 6.55 mm to (133.8, 114.0)
- moved TP106 6.55 mm to (133.8, 92.3)
- moved TP126 6.55 mm to (133.8, 59.6)
- moved TP108 6.55 mm to (133.8, 81.4)
- moved TP104 6.53 mm to (133.8, 103.2)
- moved J23 5.01 mm to (123.4, 61.2)
Connections:
- D1 pad 1: GND -> Net-(D1-Pad1)
- D10 pad 1: GND -> Net-(D10-Pad1)
- D11 pad 1: GND -> Net-(D11-Pad1)
- D12 pad 1: GND -> Net-(D12-Pad1)
- D13 pad 1: GND -> Net-(D1-Pad1)
- D14 pad 1: GND -> Net-(D1-Pad1)
- D15 pad 1: GND -> Net-(D10-Pad1)
- D16 pad 1: GND -> Net-(D10-Pad1)
- D17 pad 1: GND -> Net-(D11-Pad1)
- D18 pad 1: GND -> Net-(D11-Pad1)
- D19 pad 1: GND -> Net-(D12-Pad1)
- D2 pad 1: GND -> Net-(D10-Pad1)
- D20 pad 1: GND -> Net-(D12-Pad1)
- D3 pad 1: GND -> Net-(D11-Pad1)
- D4 pad 1: GND -> Net-(D12-Pad1)
- D5 pad 1: GND -> Net-(D1-Pad1)
- D6 pad 1: GND -> Net-(D10-Pad1)
- D7 pad 1: GND -> Net-(D11-Pad1)
- D8 pad 1: GND -> Net-(D12-Pad1)
- D9 pad 1: GND -> Net-(D1-Pad1)
- J26 pad 2: (no net) -> Net-(J26-Pad2)
- J26 pad 3: (no net) -> Net-(J26-Pad3)
- J26 pad 4: (no net) -> Net-(J26-Pad4)
- SW1 pad 3: (no net) -> Net-(SW1-Pad3)
- U2 pad 13: (no net) -> Net-(U2-Pad13)
Routing:
- net Net-(J21-Pad4): track 17.3 -> 5.44 mm
- net TEST6: track 48.0 -> 37.0 mm
- net Net-(J22-Pad4): track 5.81 -> 0.00 mm, vias 0 -> 1
- net Net-(J18-Pad4): track 5.81 -> 0.00 mm, vias 0 -> 1
- net Net-(J17-Pad4): track 5.81 -> 0.00 mm, vias 0 -> 1
- net Net-(J20-Pad4): track 5.77 -> 0.00 mm, vias 0 -> 1
- net Net-(J19-Pad4): track 5.77 -> 0.00 mm, vias 0 -> 1
- net Net-(D115-Pad1): track 1.74 -> 0.00 mm
- net +3V3: track 13.3 -> 11.9 mm, vias 6 -> 11
