File: usb-solder/usb-solder.kicad_pcb (KiCad board)
At the start: 4 copper layers, 100 x 100 mm, 313 parts, among them J1 USB_B_Micro, J10 USB_B_Micro, J11 USB_B_Micro, J12 USB_B_Micro, J13 USB_B_Micro, J14 USB_B_Micro, J15 USB_B_Micro, J16 USB_B_Micro, J17 USB_B_Micro, J18 USB_B_Micro, J19 USB_B_Micro, J2 USB_B_Micro, J20 USB_B_Micro, J21 USB_B_Micro, J22 USB_B_Micro, J23 USB_A, J24 Conn_01x02_Male, J25 Barrel_Jack_Switch, J26 USB_B_Micro, J27 Conn_01x07_Male, J3 USB_B_Micro, J4 USB_B_Micro, J5 USB_B_Micro, J6 USB_B_Micro, J7 USB_B_Micro, J8 USB_B_Micro, J9 USB_B_Micro, SW1 SW_SPDT, U1 555, U2 74HC164, U3 4072, U4 74AHC1G04, U5 AP1117-33

Commit message: script
Routing:
- net TEST6: track 37.0 -> 0.00 mm
- net Net-(R4-Pad1): track 36.4 -> 0.00 mm
- net Net-(R5-Pad1): track 32.9 -> 0.00 mm
- net TEST5: track 32.3 -> 0.00 mm
- net Net-(U1-Pad3): track 31.3 -> 0.00 mm
- net TEST3: track 31.3 -> 0.00 mm
- net TEST2: track 31.0 -> 0.00 mm
- net TEST1: track 31.0 -> 0.00 mm
- net Net-(R3-Pad1): track 25.4 -> 0.00 mm
- net Net-(R8-Pad1): track 25.4 -> 0.00 mm, vias 2 -> 0
- net Net-(R9-Pad1): track 23.6 -> 0.00 mm
- net Net-(R7-Pad1): track 22.7 -> 0.00 mm
- net Net-(R6-Pad1): track 21.7 -> 0.00 mm, vias 2 -> 0
- net Net-(U2-Pad1): track 13.1 -> 0.00 mm
- net Net-(U3-Pad13): track 12.9 -> 0.00 mm
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
Commit message: parts
Parts:
- added D121: ledred, LED_SMD:LED_0603_1608Metric, F.Cu at (18.3, 57.3)
- added D122: ledred, LED_SMD:LED_0603_1608Metric, F.Cu at (18.3, 59.9)
- added D123: ledred, LED_SMD:LED_0603_1608Metric, F.Cu at (22.3, 57.3)
- added D124: ledred, LED_SMD:LED_0603_1608Metric, F.Cu at (18.3, 62.5)
- added D125: ledred, LED_SMD:LED_0603_1608Metric, F.Cu at (22.3, 59.9)
- added D126: ledred, LED_SMD:LED_0603_1608Metric, F.Cu at (26.4, 57.3)
- added D127: ledred, LED_SMD:LED_0603_1608Metric, F.Cu at (18.3, 65.1)
- added D128: ledred, LED_SMD:LED_0603_1608Metric, F.Cu at (22.3, 62.5)
- added D129: ledred, LED_SMD:LED_0603_1608Metric, F.Cu at (26.4, 59.9)
- added D130: ledred, LED_SMD:LED_0603_1608Metric, F.Cu at (18.3, 67.7)
- added D131: ledred, LED_SMD:LED_0603_1608Metric, F.Cu at (30.4, 57.3)
- added D132: ledred, LED_SMD:LED_0603_1608Metric, F.Cu at (22.3, 65.1)
- added D133: ledred, LED_SMD:LED_0603_1608Metric, F.Cu at (26.4, 62.5)
- added D134: ledred, LED_SMD:LED_0603_1608Metric, F.Cu at (30.4, 59.9)
- added D135: ledred, LED_SMD:LED_0603_1608Metric, F.Cu at (22.3, 67.7)
- added D136: ledred, LED_SMD:LED_0603_1608Metric, F.Cu at (34.5, 57.3)
- added R16: 10k, Resistor_SMD:R_0402_1005Metric, F.Cu at (25.8, 64.8)
- added R17: 10k, Resistor_SMD:R_0402_1005Metric, F.Cu at (29.8, 62.2)
- added R18: 10k, Resistor_SMD:R_0402_1005Metric, F.Cu at (33.9, 59.6)
- added R19: 10k, Resistor_SMD:R_0402_1005Metric, F.Cu at (28.7, 64.8)
- added R20: 10k, Resistor_SMD:R_0402_1005Metric, F.Cu at (25.8, 66.8)
- added R21: 10k, Resistor_SMD:R_0402_1005Metric, F.Cu at (37.9, 57.0)
- added R22: 10k, Resistor_SMD:R_0402_1005Metric, F.Cu at (32.8, 62.2)
- added R23: 10k, Resistor_SMD:R_0402_1005Metric, F.Cu at (28.7, 66.8)
- added R24: 10k, Resistor_SMD:R_0402_1005Metric, F.Cu at (36.8, 59.6)
- added R25: 10k, Resistor_SMD:R_0402_1005Metric, F.Cu at (31.6, 64.2)
- added R26: 10k, Resistor_SMD:R_0402_1005Metric, F.Cu at (31.6, 66.2)
- added R27: 10k, Resistor_SMD:R_0402_1005Metric, F.Cu at (35.7, 61.6)
- added R28: 10k, Resistor_SMD:R_0402_1005Metric, F.Cu at (35.7, 63.6)
- added R29: 10k, Resistor_SMD:R_0402_1005Metric, F.Cu at (31.6, 68.2)
- added R30: 10k, Resistor_SMD:R_0402_1005Metric, F.Cu at (34.5, 65.6)
- added R31: 10k, Resistor_SMD:R_0402_1005Metric, F.Cu at (34.5, 67.6)
Connections:
- D1 pad 1: Net-(D1-Pad1) -> GND
- D10 pad 1: Net-(D10-Pad1) -> GND
- D11 pad 1: Net-(D11-Pad1) -> GND
- D12 pad 1: Net-(D12-Pad1) -> GND
- D13 pad 1: Net-(D1-Pad1) -> GND
- D14 pad 1: Net-(D1-Pad1) -> GND
- D15 pad 1: Net-(D10-Pad1) -> GND
- D16 pad 1: Net-(D10-Pad1) -> GND
- D17 pad 1: Net-(D11-Pad1) -> GND
- D18 pad 1: Net-(D11-Pad1) -> GND
- D19 pad 1: Net-(D12-Pad1) -> GND
- D2 pad 1: Net-(D10-Pad1) -> GND
- D20 pad 1: Net-(D12-Pad1) -> GND
- D3 pad 1: Net-(D11-Pad1) -> GND
- D4 pad 1: Net-(D12-Pad1) -> GND
- D5 pad 1: Net-(D1-Pad1) -> GND
- D6 pad 1: Net-(D10-Pad1) -> GND
- D7 pad 1: Net-(D11-Pad1) -> GND
- D8 pad 1: Net-(D12-Pad1) -> GND
- D9 pad 1: Net-(D1-Pad1) -> GND

Commit message: id
Parts:
- removed D134, D62, D66, D70, D75, D76: ledred, LED_SMD:LED_0603_1608Metric
- removed J14: USB_B_Micro, Connector_USB:USB_Micro-B_Molex-105017-0001
- removed R29: 10k, Resistor_SMD:R_0402_1005Metric
- removed TP74, TP79, TP80, TP86, TP90, TP94: TestPoint, TestPoint:TestPoint_Pad_D1.0mm
- moved D135 132.8 mm to (133.8, 140.0), turned to 270 degrees
- moved R30 122.6 mm to (133.8, 137.6)
- moved D136 122.5 mm to (133.8, 129.1), turned to 270 degrees
- moved D133 121.6 mm to (124.9, 133.8), turned to 180 degrees
- moved R31 115.5 mm to (133.8, 126.7)
- moved R28 115.4 mm to (127.3, 133.8), turned to 270 degrees
- moved D132 112.7 mm to (111.7, 133.8), turned to 180 degrees
- moved R27 106.5 mm to (114.0, 133.8), turned to 270 degrees
- moved D131 102.2 mm to (98.2, 133.8), turned to 180 degrees
- moved R26 96.5 mm to (100.5, 133.8), turned to 270 degrees
- moved D130 93.8 mm to (84.8, 133.8), turned to 180 degrees
- moved R25 89.0 mm to (87.2, 133.8), turned to 270 degrees
- moved D129 86.6 mm to (71.5, 133.8), turned to 180 degrees
- moved D128 85.9 mm to (66.2, 136.3), turned to 90 degrees
- moved R24 82.9 mm to (73.9, 133.8), turned to 270 degrees
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Connections:
- J26 pad 2: Net-(J26-Pad2) -> (no net)
- J26 pad 3: Net-(J26-Pad3) -> (no net)
- J26 pad 4: Net-(J26-Pad4) -> (no net)
- SW1 pad 3: Net-(SW1-Pad3) -> (no net)
- U2 pad 13: Net-(U2-Pad13) -> (no net)
Routing:
- net +3V3: track 0.00 -> 29.6 mm, vias 6 -> 21
- net Net-(D76-Pad2): track 21.1 -> 0.00 mm
- net Net-(J18-Pad4): track 0.00 -> 17.5 mm, vias 1 -> 2
- net Net-(J17-Pad4): track 0.00 -> 17.3 mm, vias 1 -> 2
- net Net-(J22-Pad4): track 0.00 -> 17.3 mm, vias 1 -> 2
- net Net-(J19-Pad4): track 0.00 -> 17.3 mm, vias 1 -> 2
- net Net-(J10-Pad4): track 5.77 -> 17.6 mm, vias 0 -> 2
- net Net-(J9-Pad4): track 5.77 -> 17.6 mm, vias 0 -> 2
- net Net-(J21-Pad4): track 5.44 -> 17.2 mm
- net Net-(J2-Pad4): track 5.73 -> 17.3 mm, vias 0 -> 2
- net Net-(J11-Pad4): track 5.77 -> 17.3 mm, vias 0 -> 2
- net Net-(J13-Pad4): track 5.77 -> 17.3 mm, vias 0 -> 2
- net Net-(J5-Pad4): track 5.73 -> 17.3 mm, vias 0 -> 2
- net Net-(J15-Pad4): track 5.81 -> 17.3 mm, vias 0 -> 2
- net Net-(J3-Pad4): track 5.73 -> 17.2 mm, vias 0 -> 2
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
Commit message: routing
Parts:
- added C9: 100n, Capacitor_SMD:C_0402_1005Metric, F.Cu at (110.0, 108.0)
- moved D111 29.3 mm to (96.9, 103.3), turned to 90 degrees
- moved R3 27.7 mm to (96.9, 100.3), turned to 270 degrees
- moved C3 25.8 mm to (100.5, 103.9)
- moved U3 19.0 mm to (102.9, 98.3), turned to 180 degrees
- moved R4 18.6 mm to (119.8, 103.8)
- moved U1 17.9 mm to (112.2, 85.1), turned to 90 degrees
- moved C2 17.7 mm to (108.3, 85.0), turned to 270 degrees
- moved C1 17.1 mm to (114.7, 82.4), turned to 90 degrees
- moved C5 16.2 mm to (109.7, 85.0), turned to 270 degrees
- moved C4 15.7 mm to (109.6, 103.8), turned to 0 degrees
- moved R5 15.2 mm to (119.8, 101.1)
- moved J27 13.8 mm to (124.7, 104.1), turned to 180 degrees
- moved C6 13.5 mm to (113.3, 80.2), turned to 0 degrees
- moved R1 13.0 mm to (109.8, 82.5), turned to 90 degrees
- moved R6 11.9 mm to (119.8, 98.4)
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Connections:
- U3 pad 10: Net-(U3-Pad1) -> Net-(R4-Pad1)
- U3 pad 11: Net-(R4-Pad1) -> Net-(R3-Pad1)
- U3 pad 12: Net-(R3-Pad1) -> Net-(U3-Pad1)
Routing:
- net +3V3: track 29.6 -> 90.4 mm, vias 21 -> 36
- net TEST6: track 0.00 -> 57.0 mm
- net TEST1: track 0.00 -> 52.9 mm
- net TEST2: track 0.00 -> 49.4 mm
- net GND: track 0.00 -> 47.5 mm, vias 0 -> 18
- net TEST3: track 0.00 -> 47.2 mm
- net TEST5: track 0.00 -> 42.8 mm
- net Net-(R4-Pad1): track 0.00 -> 23.6 mm
- net Net-(R5-Pad1): track 0.00 -> 22.9 mm
- net VIN: track 0.00 -> 22.5 mm
- net Net-(R3-Pad1): track 0.00 -> 20.1 mm
- net Net-(R8-Pad1): track 0.00 -> 19.2 mm, vias 0 -> 2
- net Net-(R9-Pad1): track 0.00 -> 17.3 mm, vias 0 -> 2
- net Net-(R7-Pad1): track 0.00 -> 16.8 mm, vias 0 -> 2
- net Net-(R6-Pad1): track 0.00 -> 16.5 mm
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- added copper zone on F.Cu, net GND
