File: usb-solder/usb-solder.kicad_pcb (KiCad board)
At the start: 4 copper layers, 100 x 100 mm, 332 parts, among them J1 USB_B_Micro, J10 USB_B_Micro, J11 USB_B_Micro, J12 USB_B_Micro, J13 USB_B_Micro, J15 USB_B_Micro, J16 USB_B_Micro, J17 USB_B_Micro, J18 USB_B_Micro, J19 USB_B_Micro, J2 USB_B_Micro, J20 USB_B_Micro, J21 USB_B_Micro, J22 USB_B_Micro, J23 USB_A, J24 Conn_01x02_Male, J25 Barrel_Jack_Switch, J26 USB_B_Micro, J27 Conn_01x07_Male, J3 USB_B_Micro, J4 USB_B_Micro, J5 USB_B_Micro, J6 USB_B_Micro, J7 USB_B_Micro, J8 USB_B_Micro, J9 USB_B_Micro, SW1 SW_SPDT, U1 555, U2 74HC164, U3 4072, U4 74AHC1G04, U5 AP1117-33

Commit message: silk
Other:
- board text added: "*"
- board text added: "-"
- board text added: "1"
- board text added: "10"
- board text added: "11"
- board text added: "12"
- board text added: "13"
- board text added: "14"
- board text added: "15"
- board text added: "16"
- board text added: "17"
- board text added: "18"
- board text added: "19"
- board text added: "2"
- board text added: "20"
- board text added: "21"
- board text added: "3"
- board text added: "4"
- board text added: "4.6 to 12 volts 100 mA"
- board text added: "5"
- board text added: "6"
- board text added: "7"
- board text added: "8"
- board text added: "9"
- board text added: "GND"
- board text added: "ON OFF"
- board text added: "OTG"
- board text added: "OTG LED shows status of pin 4 on = OTG cable"
- board text added: "TEST SIGNAL OUTPUT"
- board text added: "Test Points"
- board text added: "USB Solder Practice 2020-12-27"
- board text added: "Use one of J24, J25, J26"
- board text added: "github.com/pacew/usb-solder"

Commit message: logo
Parts:
- added G***: LOGO, pace:aalogo, F.Cu at (85.2, 91.0)
Other:
- board text added: "4.6 to 12 volts"
- board text removed: "4.6 to 12 volts 100 mA"

Commit message: v1
Parts:
- removed G***: LOGO, pace:aalogo
- removed R9: 10k, Resistor_SMD:R_0402_1005Metric
- J27: value Conn_01x07_Male -> Conn_01x06_Male; footprint Connector_PinHeader_2.54mm:PinHeader_1x07_P2.54mm_Vertical -> Connector_PinHeader_2.54mm:PinHeader_1x06_P2.54mm_Vertical
- moved R8 2.88 mm to (119.8, 93.2)
- moved R7 2.69 mm to (119.8, 95.8)
- moved J27 0.14 mm to (124.8, 104.2)
Connections:
- J27 pad 4: TEST4 -> TEST5
- J27 pad 5: TEST5 -> TEST6
- J27 pad 6: TEST6 -> GND
- U2 pad 12: Net-(R9-Pad1) -> (no net)
- U3 pad 2: Net-(R9-Pad1) -> GND
Routing:
- net Net-(R9-Pad1): track 17.3 -> 0.00 mm, vias 2 -> 0
- net TEST4: track 5.04 -> 0.00 mm
- net TEST5: track 42.8 -> 46.0 mm
- net TEST6: track 57.0 -> 59.8 mm
- net GND: track 47.5 -> 49.4 mm, vias 18 -> 19
- net Net-(R7-Pad1): track 16.8 -> 15.9 mm
Other:
- board text added: "Power input"
- board text removed: "-"

Commit message: v1
Parts:
- added LOGO1: aalogo, pace:aalogo, F.Cu at (86.2, 91.5)
