File: usb-solder/usb-solder.sch (KiCad schematic (older format))
At the start: 187 parts, among them J1 USB_B_Micro, J10 USB_B_Micro, J11 USB_B_Micro, J12 USB_B_Micro, J13 USB_B_Micro, J14 USB_B_Micro, J15 USB_B_Micro, J16 USB_B_Micro, J17 USB_B_Micro, J18 USB_B_Micro, J19 Barrel_Jack_Switch, J2 USB_B_Micro, J20 Conn_01x02_Male, J21 USB_B_Micro, J22 USB_B_Micro, J23 USB_B_Micro, J24 USB_A, J25 USB_B_Micro, J26 USB_B_Micro, J27 USB_B_Micro, J3 USB_B_Micro, J4 USB_B_Micro, J5 USB_B_Micro, J6 USB_B_Micro, J7 USB_B_Micro, J8 USB_B_Micro, J9 USB_B_Micro, U1 555, U2 74HC164, U3 4072, U4 74HC04, U5 AP1117-33

Commit message: new
Parts:
- removed D112, D113, D114, D115, D116, D117, D118, D119, D120, D121, D122, D123, D124, D125, D126, D127, D128, D129, D130, D131, D132, D133, D134, D135, D136, D137, D138, D139, D140, D141, D142, D143, D144, D145: ledred, LED_SMD:LED_0603_1608Metric, symbol pace:ledred
- removed J23, J25, J27: USB_B_Micro, Connector_USB:USB_Micro-B_Molex-105017-0001, symbol pace:USB_B_Micro
- added C5: 100n, Capacitor_SMD:C_0402_1005Metric, symbol pace:100n
- added D109: ledred, LED_SMD:LED_0603_1608Metric, symbol pace:ledred
- added D112, D114: SS210, Diode_SMD:D_SMA, symbol pace:SS210
- added H1, H2, H3, H4: MountingHole, MountingHole:MountingHole_3.5mm, symbol Mechanical:MountingHole
- added J19, J20: USB_B_Micro, Connector_USB:USB_Micro-B_Molex-105017-0001, symbol pace:USB_B_Micro
- added J27: Conn_01x07_Male, Connector_PinHeader_2.54mm:PinHeader_1x07_P2.54mm_Vertical, symbol Connector:Conn_01x07_Male
- added R3, R4, R5, R6, R7, R8, R9: 10k, Resistor_SMD:R_0402_1005Metric, symbol pace:10k
- added SW1: SW_SPDT, pace:Switch_Toggle_ATE1D-2M3-10-Z, symbol pace:SW_SPDT
- added TP1, TP10, TP100, TP101, TP102, TP103, TP104, TP105, TP106, TP107, TP108, TP109, TP11, TP110, TP111, TP112, TP113, TP114, TP115, TP116, TP117, TP118, TP119, TP12, TP120, TP121, TP122, TP123, TP124, TP125, TP126, TP127, TP128, TP129, TP13, TP130, TP131, TP132, TP14, TP15, TP16, TP17, TP18, TP19, TP2, TP20, TP21, TP22, TP23, TP24, TP25, TP26, TP27, TP28, TP29, TP3, TP30, TP31, TP32, TP33, TP34, TP35, TP36, TP37, TP38, TP39, TP4, TP40, TP41, TP42, TP43, TP44, TP45, TP46, TP47, TP48, TP49, TP5, TP50, TP51, TP52, TP53, TP54, TP55, TP56, TP57, TP58, TP59, TP6, TP60, TP61, TP62, TP63, TP64, TP65, TP66, TP67, TP68, TP69, TP7, TP70, TP71, TP72, TP73, TP74, TP75, TP76, TP77, TP78, TP79, TP8, TP80, TP81, TP82, TP83, TP84, TP85, TP86, TP87, TP88, TP89, TP9, TP90, TP91, TP92, TP93, TP94, TP95, TP96, TP97, TP98, TP99: TestPoint, TestPoint:TestPoint_Pad_D1.0mm, symbol pace:TestPoint
- renumbered C5 to C6, C6 to C7, C7 to C8, D109 to D113, J24 to J23, J20 to J24, J19 to J25
Connections:
- net +3V3: now also C5.1
- net GND: now also J26.5 (GND), C5.2, D109.1 (K), J27.7 (Pin_7); no longer U3.12
- net at D1.2 (A), J1.1 (VBUS): now also TP5.1
- net at J1.2 (D-): now also D13.2 (A), TP21.1; no longer D2.2 (A)
- net at J1.3 (D+): now also D9.2 (A), TP17.1; no longer D13.2 (A)
- net at J1.4 (ID): now also TP6.1; no longer D14.2 (A)
- net at J1.5 (GND): now also D5.2 (A), TP13.1; no longer D3.2 (A)
- net at J1.6 (Shield): now also D14.2 (A), TP1.1; no longer D15.2 (A)
- net at J2.1 (VBUS): now also D2.2 (A), TP7.1; no longer D4.2 (A)
- net at J2.2 (D-): now also D15.2 (A), TP22.1; no longer D5.2 (A)
- net at J2.3 (D+): now also D10.2 (A), TP18.1; no longer D16.2 (A)
- net at J2.4 (ID): now also TP8.1; no longer D17.2 (A)
- net at D6.2 (A), J2.5 (GND): now also TP14.1
- net at J2.6 (Shield): now also D16.2 (A), TP2.1; no longer D18.2 (A)
- net at J3.1 (VBUS): now also D3.2 (A), TP9.1; no longer D7.2 (A)
- net at J3.2 (D-): now also D17.2 (A), TP23.1; no longer D8.2 (A)
- net at J3.3 (D+): now also D11.2 (A), TP19.1; no longer D19.2 (A)
- net at J3.4 (ID): now also TP10.1; no longer D20.2 (A)
- net at J3.5 (GND): now also D7.2 (A), TP15.1; no longer D9.2 (A)
- net at J3.6 (Shield): now also D18.2 (A), TP3.1; no longer D21.2 (A)
- net at J4.1 (VBUS): now also D4.2 (A), TP11.1; no longer D10.2 (A)
- net at J4.2 (D-): now also D19.2 (A), TP24.1; no longer D11.2 (A)
- net at J4.3 (D+): now also D12.2 (A), TP20.1; no longer D22.2 (A)
- net at J4.4 (ID): now also TP12.1; no longer D23.2 (A)
- net at J4.5 (GND): now also D8.2 (A), TP16.1; no longer D12.2 (A)
- net at J4.6 (Shield): now also D20.2 (A), TP4.1; no longer D24.2 (A)
- net at D58.2 (A): now also J11.6 (Shield), TP51.1; no longer J12.1 (VBUS)
- net at D59.2 (A), J12.2 (D-): now also TP72.1
- net at J12.3 (D+): now also D52.2 (A), TP68.1; no longer D70.2 (A)
- net at J12.4 (ID): now also TP60.1; no longer D71.2 (A)
- net at J12.5 (GND): now also D48.2 (A), TP64.1; no longer D60.2 (A)
- net at J12.6 (Shield): now also D60.2 (A), TP52.1; no longer D72.2 (A)
- net at D34.2 (A): now also J5.6 (Shield), TP25.1; no longer J8.1 (VBUS)
- net at D35.2 (A): now also J6.2 (D-), TP46.1; no longer J8.2 (D-)
- net at J8.3 (D+): now also D32.2 (A), TP44.1; no longer D46.2 (A)
- net at J8.4 (ID): now also TP36.1; no longer D47.2 (A)
- net at D36.2 (A): now also J6.6 (Shield), TP26.1; no longer J8.5 (GND)
- net at J8.6 (Shield): now also D40.2 (A), TP28.1; no longer D48.2 (A)
- net at J5.1 (VBUS): now also D21.2 (A), TP29.1; no longer D25.2 (A)
- net at J5.2 (D-): now also D33.2 (A), TP45.1; no longer D26.2 (A)
- net at J5.3 (D+): now also D29.2 (A), TP41.1; no longer D37.2 (A)
- net at J5.4 (ID): now also TP30.1; no longer D38.2 (A)
- net at J5.5 (GND): now also D25.2 (A), TP37.1; no longer D27.2 (A)
- net at D39.2 (A): now also J8.2 (D-), TP48.1; no longer J5.6 (Shield)
- net at J6.1 (VBUS): now also D22.2 (A), TP31.1; no longer D28.2 (A)
- net at J6.3 (D+): now also D30.2 (A), TP42.1; no longer D40.2 (A)
- net at J6.4 (ID): now also TP32.1; no longer D41.2 (A)
- net at J6.5 (GND): now also D26.2 (A), TP38.1; no longer D30.2 (A)
- net at D42.2 (A): now also J10.1 (VBUS), TP55.1; no longer J6.6 (Shield)
- net at J7.1 (VBUS): now also D23.2 (A), TP33.1; no longer D31.2 (A)
- net at J7.2 (D-): now also D37.2 (A), TP47.1; no longer D32.2 (A)
- net at J7.3 (D+): now also D31.2 (A), TP43.1; no longer D43.2 (A)
- net at J7.4 (ID): now also TP34.1; no longer D44.2 (A)
- net at J7.5 (GND): now also D27.2 (A), TP39.1; no longer D33.2 (A)
- net at J7.6 (Shield): now also D38.2 (A), TP27.1; no longer D45.2 (A)
- net at J16.1 (VBUS): now also D64.2 (A), TP83.1; no longer D91.2 (A)
- net at J16.2 (D-): now also D79.2 (A), TP96.1; no longer D92.2 (A)
- net at J16.3 (D+): now also D72.2 (A), TP92.1; no longer D100.2 (A)
- net at J16.4 (ID): now also TP84.1; no longer D101.2 (A)
- net at J16.5 (GND): now also D68.2 (A), TP88.1; no longer D93.2 (A)
- net at J16.6 (Shield): now also D80.2 (A), TP76.1; no longer D102.2 (A)
- net at J17.1 (VBUS): now also D81.2 (A), TP101.1; no longer D94.2 (A)
- net at J17.2 (D-): now also D93.2 (A), TP117.1; no longer D95.2 (A)
- net at J17.3 (D+): now also D89.2 (A), TP113.1; no longer D103.2 (A)
- net at J17.4 (ID): now also TP102.1; no longer D104.2 (A)
- net at J17.5 (GND): now also D85.2 (A), TP109.1; no longer D96.2 (A)
- net at J17.6 (Shield): now also D94.2 (A), TP97.1; no longer D105.2 (A)
- net at J18.1 (VBUS): now also D82.2 (A), TP103.1; no longer D97.2 (A)
- net at J18.2 (D-): now also D95.2 (A), TP118.1; no longer D98.2 (A)
- net at J18.3 (D+): now also D90.2 (A), TP114.1; no longer D106.2 (A)
- net at J18.4 (ID): now also TP104.1; no longer D107.2 (A)
- net at J18.5 (GND): now also D86.2 (A), TP110.1; no longer D99.2 (A)
- net at J18.6 (Shield): now also D96.2 (A), TP98.1; no longer D108.2 (A)
- net at J9.1 (VBUS): now also D41.2 (A), TP53.1; no longer D49.2 (A)
- net at J9.2 (D-): now also D53.2 (A), TP69.1; no longer D50.2 (A)
- net at J9.3 (D+): now also D49.2 (A), TP65.1; no longer D61.2 (A)
- net at J9.4 (ID): now also TP54.1; no longer D62.2 (A)
- net at J9.5 (GND): now also D45.2 (A), TP61.1; no longer D51.2 (A)
- net at J9.6 (Shield): now also D54.2 (A), TP49.1; no longer D63.2 (A)
- net at J10.2 (D-): now also D55.2 (A), TP70.1; no longer D53.2 (A)
- net at J10.3 (D+): now also D50.2 (A), TP66.1; no longer D64.2 (A)
- net at J10.4 (ID): now also TP56.1; no longer D65.2 (A)
- net at J10.5 (GND): now also D46.2 (A), TP62.1; no longer D54.2 (A)
- net at J10.6 (Shield): now also D56.2 (A), TP50.1; no longer D66.2 (A)
- net at J11.1 (VBUS): now also D43.2 (A), TP57.1; no longer D55.2 (A)
- net at J11.2 (D-): now also D57.2 (A), TP71.1; no longer D56.2 (A)
- net at J11.3 (D+): now also D51.2 (A), TP67.1; no longer D67.2 (A)
- net at J11.4 (ID): now also TP58.1; no longer D68.2 (A)
- net at J11.5 (GND): now also D47.2 (A), TP63.1; no longer D57.2 (A)
- net at D69.2 (A): now also J13.3 (D+), TP89.1; no longer J11.6 (Shield)
- net at J21.1 (VBUS): now also D101.2 (A), TP123.1; no longer D110.2 (A)
- net at J21.2 (D-): now also D107.2 (A), TP131.1; no longer D111.2 (A)
- net at J21.3 (D+): now also D105.2 (A), TP129.1
- net at J21.4 (ID): now also TP124.1
- net at J21.5 (GND): now also D103.2 (A), TP127.1
- net at J21.6 (Shield): now also D108.2 (A), TP121.1
- net at J22.1 (VBUS): now also D102.2 (A), TP125.1
- net at J22.2 (D-): now also D109.2 (A), TP132.1
- net at J22.3 (D+): now also D106.2 (A), TP130.1
- net at J22.4 (ID): now also TP126.1
- net at J22.5 (GND): now also D104.2 (A), TP128.1
- net at J22.6 (Shield): now also D110.2 (A), TP122.1
- net at J13.1 (VBUS): now also D61.2 (A), TP77.1; no longer D73.2 (A)
- net at J13.2 (D-): now also D73.2 (A), TP93.1; no longer D74.2 (A)
- net at J13.4 (ID): now also TP78.1; no longer D83.2 (A)
- net at J13.5 (GND): now also D65.2 (A), TP85.1; no longer D75.2 (A)
- net at J13.6 (Shield): now also D74.2 (A), TP73.1; no longer D84.2 (A)
- net at J14.1 (VBUS): now also D62.2 (A), TP79.1; no longer D76.2 (A)
- net at J14.2 (D-): now also D75.2 (A), TP94.1; no longer D77.2 (A)
- net at J14.3 (D+): now also D70.2 (A), TP90.1; no longer D85.2 (A)
- net at J14.4 (ID): now also TP80.1; no longer D86.2 (A)
- net at J14.5 (GND): now also D66.2 (A), TP86.1; no longer D78.2 (A)
- net at J14.6 (Shield): now also D76.2 (A), TP74.1; no longer D87.2 (A)
- net at J15.1 (VBUS): now also D63.2 (A), TP81.1; no longer D79.2 (A)
- net at J15.2 (D-): now also D77.2 (A), TP95.1; no longer D80.2 (A)
- net at J15.3 (D+): now also D71.2 (A), TP91.1; no longer D88.2 (A)
- net at J15.4 (ID): now also TP82.1; no longer D89.2 (A)
- net at J15.5 (GND): now also D67.2 (A), TP87.1; no longer D81.2 (A)
- net at J15.6 (Shield): now also D78.2 (A), TP75.1; no longer D90.2 (A)
- net at J26.1 (VBUS): now also D114.2 (A)
- net LAST: now reaches U2.12 (Q6)
- net LAST: now also U3.12, R9.1
- net at U2.6 (Q3), U3.5: now also R6.1
- net at C7.1, U5.3 (VI): now also F1.1; no longer D113.1 (K)
- net at D113.2 (A): now also J25.1; no longer F1.1
- net TEST_DM: no longer names the net of U2.5 (Q2), U3.4
- net TEST_DM: now also R5.1; no longer J23.3 (D+)
- net TEST_DP: no longer names the net of U2.4 (Q1), U3.3
- net TEST_DP: now also R4.1; no longer J23.2 (D-)
- net TEST_GND: no longer names the net of U2.10 (Q4), U3.10
- net TEST_GND: now also R7.1; no longer J23.4 (GND)
- net TEST_SHIELD: no longer names the net of U2.11 (Q5), U3.11
- net TEST_SHIELD: now also R8.1; no longer J23.5 (Shield)
- net TEST_VBUS: no longer names the net of U2.3 (Q0), U3.2
- net TEST_VBUS: now also R3.1; no longer J23.1 (VBUS)
- new net: D24.2 (A), J8.1 (VBUS), TP35.1
- new net: D28.2 (A), J8.5 (GND), TP40.1
- new net: D44.2 (A), J12.1 (VBUS), TP59.1
- new net: D83.2 (A), J19.1 (VBUS), TP105.1
- new net: D97.2 (A), J19.2 (D-), TP119.1
- new net: D91.2 (A), J19.3 (D+), TP115.1
- new net: J19.4 (ID), TP106.1
- new net: D87.2 (A), J19.5 (GND), TP111.1
- new net: D98.2 (A), J19.6 (Shield), TP99.1
- new net: D84.2 (A), J20.1 (VBUS), TP107.1
- new net: D99.2 (A), J20.2 (D-), TP120.1
- new net: D92.2 (A), J20.3 (D+), TP116.1
- new net: J20.4 (ID), TP108.1
- new net: D88.2 (A), J20.5 (GND), TP112.1
- new net: D100.2 (A), J20.6 (Shield), TP100.1
- new net: D112.2 (A), J24.1 (Pin_1)
- new net: D111.2 (A), R9.2
- new net: F1.2, SW1.1 (A)
- new net TEST1: J23.1 (VBUS), J27.1 (Pin_1), R3.2
- new net TEST2: J23.2 (D-), J27.2 (Pin_2), R4.2
- new net TEST3: J23.3 (D+), J27.3 (Pin_3), R5.2
- new net TEST4: J27.4 (Pin_4), R8.2
- new net TEST5: J23.4 (GND), J27.5 (Pin_5), R6.2
- new net TEST6: J23.5 (Shield), J27.6 (Pin_6), R7.2
- new net VIN: D112.1 (K), D113.1 (K), D114.1 (K), SW1.2 (B)
- no-connect marks 2 -> 7
Other:
- note added: "200 millisec period clock"
- note added: "ID pin (TEST4) out of order since it\nis not present on a standard cable"
- note added: "pin 4 on the USB A connector\ngoes to pin 5 on the USB B"
- note removed: "slow clock - period 207 milliseconds"
- note removed: "what do do about ID?\n"
- moved on the sheet: C1, C7, C8, D113, F1, J23, J24, J25, U5

Commit message: routing
Parts:
- removed U4: 74HC04, Package_SO:SOIC-14_3.9x8.7mm_P1.27mm, symbol pace:74HC04
- added unit 3 of U3
- added U4: 74AHC1G04, Package_TO_SOT_SMD:SOT-353_SC-70-5, symbol pace:74AHC1G04
Connections:
- net +3V3: now also U3.14, U4.5 (VCC)
- net GND: now also U3.7, U4.3 (GND)
- net TEST1: now also R4.2; no longer R3.2
- net TEST2: now also R5.2; no longer R4.2
- net TEST3: now also R6.2; no longer R5.2
- net TEST4: now also R9.2; no longer R8.2
- net TEST5: now also R7.2; no longer R6.2
- net TEST6: now also R8.2; no longer R7.2
- net at U3.13: now also U4.2
- net at U2.1 (DSA), U2.2 (DSB): now also U4.4
- net at R7.1, U2.10 (Q4): now also U3.4; no longer U3.10
- net at R8.1, U2.11 (Q5): now also U3.3; no longer U3.11
- net at R3.1, U2.3 (Q0): now also U3.12; no longer U3.2
- net at R4.1, U2.4 (Q1): now also U3.11; no longer U3.3
- net at R5.1, U2.5 (Q2): now also U3.9; no longer U3.4
- net at U3.1: now also U3.10; no longer U3.9
- net SYNC: now reaches D111.2 (A)
- net SYNC: now also R3.2; no longer R9.2
- net LAST: no longer names the net of R9.1, U2.12 (Q6)
- net LAST: now also U3.2; no longer U3.12
Other:
- moved on the sheet: R3, R4, R5, R6, R7, R8, U3A, U3B

Commit message: lib
Parts:
- removed H1, H2, H3, H4: MountingHole, MountingHole:MountingHole_3.5mm, symbol Mechanical:MountingHole
- added H1, H2, H3, H4: MountingHole_Pad, MountingHole:MountingHole_3.2mm_M3_Pad, symbol pace:MountingHole_Pad
- J24: symbol Connector:Conn_01x02_Male -> pace:Conn_01x02_Male
- J27: symbol Connector:Conn_01x07_Male -> pace:Conn_01x07_Male
Connections:
- net GND: now also H1.1, H2.1, H3.1, H4.1

Commit message: id
Parts:
- added D115: ledred, LED_SMD:LED_0603_1608Metric, symbol pace:ledred
- added R10: 10k, Resistor_SMD:R_0402_1005Metric, symbol pace:10k
Connections:
- net +3V3: now also D115.2 (A)
- net at J21.4 (ID), TP124.1: now also R10.2
- new net: D115.1 (K), R10.1
- no-connect marks 7 -> 6
Changed lines of the file:
@@
-$EndComp
-$Comp
-L pace:TestPoint TP131
-U 1 1 600B0D28
-P 7900 1250
-F 0 "TP131" H 7958 1322 50  0001 L CNN
-F 1 "TestPoint" H 7900 1450 50  0001 C CNN
-F 2 "TestPoint:TestPoint_Pad_D1.0mm" H 8100 1250 50  0001 C CNN
-F 3 "~" H 8100 1250 50  0001 C CNN
-	1    7900 1250
-	1    0    0    -1
 $EndComp
 $Comp
 L pace:ledred D107
 U 1 1 600B0D2F
-P 8000 1250
-F 0 "D107" H 8000 1150 50  0001 C CNN
-F 1 "ledred" H 8000 1394 50  0001 C CNN
-F 2 "LED_SMD:LED_0603_1608Metric" V 8000 1250 50  0001 C CNN
-F 3 "https://datasheet.lcsc.com/szlcsc/Hubei-KENTO-Elec-KT-0603R_C2286.pdf" V 8000 1250 50  0001 C CNN
-F 4 "C2286" H 8000 1250 50  0001 C CNN "LCSC"
-	1    8000 1250
+P 8000 1150
+F 0 "D107" H 8000 1050 50  0001 C CNN
+F 1 "ledred" H 8000 1294 50  0001 C CNN
+F 2 "LED_SMD:LED_0603_1608Metric" V 8000 1150 50  0001 C CNN
+F 3 "https://datasheet.lcsc.com/szlcsc/Hubei-KENTO-Elec-KT-0603R_C2286.pdf" V 8000 1150 50  0001 C CNN
+F 4 "C2286" H 8000 1150 50  0001 C CNN "LCSC"
+	1    8000 1150
 	-1   0    0    1
 $EndComp
@@
 L pace:TestPoint TP124
 U 1 1 600B0D35
-P 7500 1250
-F 0 "TP124" H 7558 1322 50  0001 L CNN
-F 1 "TestPoint" H 7500 1450 50  0001 C CNN
-F 2 "TestPoint:TestPoint_Pad_D1.0mm" H 7700 1250 50  0001 C CNN
-F 3 "~" H 7700 1250 50  0001 C CNN
-	1    7500 1250
+P 8250 1250
+F 0 "TP124" H 8308 1322 50  0001 L CNN
+F 1 "TestPoint" H 8250 1450 50  0001 C CNN
+F 2 "TestPoint:TestPoint_Pad_D1.0mm" H 8450 1250 50  0001 C CNN
+F 3 "~" H 8450 1250 50  0001 C CNN
+	1    8250 1250
 	-1   0    0    1
 $EndComp
@@
 	7500 1050 7700 1050
 Connection ~ 7700 1050
-Wire Wire Line
-	7500 1150 7700 1150
-Wire Wire Line
-	7700 1150 7700 1250
-Wire Wire Line
-	7700 1250 7900 1250
-Connection ~ 7900 1250
+Connection ~ 7900 1150
 $Comp
 L pace:ledred D103
@@
 	8100 850  8100 1050
 Connection ~ 8100 1500
-Connection ~ 8100 1250
-Wire Wire Line
-	8100 1250 8100 1350
+Connection ~ 8100 1150
+Wire Wire Line
+	8100 1150 8100 1350
 Wire Wire Line
 	7900 1050 8100 1050
 Connection ~ 8100 1050
 Wire Wire Line
-	8100 1050 8100 1250
+	8100 1050 8100 1150
 Wire Wire Line
 	7800 1350 8100 1350
@@
 $EndComp
 NoConn ~ 8550 4350
-NoConn ~ 750  1000
 $Comp
 L pace:10k R9
@@
 	1    0    0    -1
 $EndComp
+$Comp
+L pace:+3.3V #PWR?
+U 1 1 5FF0EE57
+P 8250 850
+F 0 "#PWR?" H 8250 700 50  0001 C CNN
+F 1 "+3.3V" H 8265 1023 50  0000 C CNN
+F 2 "" H 8250 850 50  0001 C CNN
+F 3 "" H 8250 850 50  0001 C CNN
+	1    8250 850
+	1    0    0    -1
+$EndComp
+$Comp
+L pace:ledred D115
+U 1 1 5FF14412
+P 8250 950
+F 0 "D115" H 8250 850 50  0001 C CNN
+F 1 "ledred" H 8250 1094 50  0001 C CNN
+F 2 "LED_SMD:LED_0603_1608Metric" V 8250 950 50  0001 C CNN
+F 3 "https://datasheet.lcsc.com/szlcsc/Hubei-KENTO-Elec-KT-0603R_C2286.pdf" V 8250 950 50  0001 C CNN
+F 4 "C2286" H 8250 950 50  0001 C CNN "LCSC"
+	1    8250 950
+	0    -1   -1   0
+$EndComp
+$Comp
+L pace:10k R10
+U 1 1 5FF2ED5D
+P 8250 1150
+F 0 "R10" V 8300 1300 50  0001 L CNN
+F 1 "10k" V 8300 900 50  0001 L CNN
+F 2 "Resistor_SMD:R_0402_1005Metric" H 8250 1150 50  0001 C CNN
+F 3 "https://datasheet.lcsc.com/szlcsc/Uniroyal-Elec-0402WGF1002TCE_C25744.pdf" H 8250 1150 50  0001 C CNN
+F 4 "C25744" H 8250 1150 50  0001 C CNN "LCSC"
+	1    8250 1150
+	1    0    0    -1
+$EndComp
+$Comp
+L pace:TestPoint TP131
+U 1 1 600B0D28
+P 7900 1150
+F 0 "TP131" H 7958 1222 50  0001 L CNN
+F 1 "TestPoint" H 7900 1350 50  0001 C CNN
+F 2 "TestPoint:TestPoint_Pad_D1.0mm" H 8100 1150 50  0001 C CNN
+F 3 "~" H 8100 1150 50  0001 C CNN
+	1    7900 1150
+	1    0    0    -1
+$EndComp
+Wire Wire Line
+	7500 1150 7900 1150
+Wire Wire Line
+	7500 1250 8250 1250
+Connection ~ 8250 1250
 $EndSCHEMATC

Commit message: id
Parts:
- added D116, D117, D118, D119, D120: ledred, LED_SMD:LED_0603_1608Metric, symbol pace:ledred
- added R11, R12, R13, R14, R15: 10k, Resistor_SMD:R_0402_1005Metric, symbol pace:10k
Connections:
- net +3V3: now also D116.2 (A), D117.2 (A), D118.2 (A), D119.2 (A), D120.2 (A)
- net GND: no longer D1.1 (K), D10.1 (K), D11.1 (K), D12.1 (K), D13.1 (K), D14.1 (K), D15.1 (K), D16.1 (K), D17.1 (K), D18.1 (K), D19.1 (K), D2.1 (K), D20.1 (K), D3.1 (K), D4.1 (K), D5.1 (K), D6.1 (K), D7.1 (K), D8.1 (K), D9.1 (K)
- net at J17.4 (ID), TP102.1: now also R11.2
- net at J18.4 (ID), TP104.1: now also R12.2
- net at J19.4 (ID), TP106.1: now also R13.2
- net at J20.4 (ID), TP108.1: now also R14.2
- net at J22.4 (ID), TP126.1: now also R15.2
- new net: D1.1 (K), D13.1 (K), D14.1 (K), D5.1 (K), D9.1 (K)
- new net: D10.1 (K), D15.1 (K), D16.1 (K), D2.1 (K), D6.1 (K)
- new net: D11.1 (K), D17.1 (K), D18.1 (K), D3.1 (K), D7.1 (K)
- new net: D12.1 (K), D19.1 (K), D20.1 (K), D4.1 (K), D8.1 (K)
- new net: D120.1 (K), R15.1
- new net: D116.1 (K), R11.1
- new net: D117.1 (K), R12.1
- new net: D118.1 (K), R13.1
- new net: D119.1 (K), R14.1
Other:
- moved on the sheet: C2, C3, C4, C5, C7, C8, D112, D113, D114, F1, J10, J11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

Commit message: id
Parts:
- added D121, D122, D123, D124, D125, D126, D127, D128, D129, D130, D131, D132, D133, D134, D135, D136: ledred, LED_SMD:LED_0603_1608Metric, symbol pace:ledred
- added R16, R17, R18, R19, R20, R21, R22, R23, R24, R25, R26, R27, R28, R29, R30, R31: 10k, Resistor_SMD:R_0402_1005Metric, symbol pace:10k
Connections:
- net +3V3: now also D121.2 (A), D122.2 (A), D123.2 (A), D124.2 (A), D125.2 (A), D126.2 (A), D127.2 (A), D128.2 (A), D129.2 (A), D130.2 (A), D131.2 (A), D132.2 (A), D133.2 (A), D134.2 (A), D135.2 (A), D136.2 (A)
- net GND: now also D1.1 (K), D10.1 (K), D11.1 (K), D12.1 (K), D13.1 (K), D14.1 (K), D15.1 (K), D16.1 (K), D17.1 (K), D18.1 (K), D19.1 (K), D2.1 (K), D20.1 (K), D3.1 (K), D4.1 (K), D5.1 (K), D6.1 (K), D7.1 (K), D8.1 (K), D9.1 (K)
- net at J1.4 (ID), TP6.1: now also R16.2
- net at J2.4 (ID), TP8.1: now also R17.2
- net at J3.4 (ID), TP10.1: now also R18.2
- net at J4.4 (ID), TP12.1: now also R19.2
- net at J5.4 (ID), TP30.1: now also R20.2
- net at J6.4 (ID), TP32.1: now also R21.2
- net at J7.4 (ID), TP34.1: now also R22.2
- net at J8.4 (ID), TP36.1: now also R23.2
- net at J9.4 (ID), TP54.1: now also R24.2
- net at J10.4 (ID), TP56.1: now also R25.2
- net at J11.4 (ID), TP58.1: now also R26.2
- net at J12.4 (ID), TP60.1: now also R27.2
- net at J13.4 (ID), TP78.1: now also R28.2
- net at J14.4 (ID), TP80.1: now also R29.2
- net at J15.4 (ID), TP82.1: now also R30.2
- net at J16.4 (ID), TP84.1: now also R31.2
- new net: D133.1 (K), R28.1
- new net: D134.1 (K), R29.1
- new net: D135.1 (K), R30.1
- new net: D136.1 (K), R31.1
- new net: D132.1 (K), R27.1
- new net: D131.1 (K), R26.1
- new net: D130.1 (K), R25.1
- new net: D129.1 (K), R24.1
- new net: D125.1 (K), R20.1
- new net: D126.1 (K), R21.1
- new net: D127.1 (K), R22.1
- new net: D128.1 (K), R23.1
- new net: D124.1 (K), R19.1
- new net: D123.1 (K), R18.1
- new net: D122.1 (K), R17.1
- new net: D121.1 (K), R16.1
