File: usb-solder/usb-solder.sch (KiCad schematic (older format))
At the start: 345 parts, among them J1 USB_B_Micro, J10 USB_B_Micro, J11 USB_B_Micro, J12 USB_B_Micro, J13 USB_B_Micro, J14 USB_B_Micro, J15 USB_B_Micro, J16 USB_B_Micro, J17 USB_B_Micro, J18 USB_B_Micro, J19 USB_B_Micro, J2 USB_B_Micro, J20 USB_B_Micro, J21 USB_B_Micro, J22 USB_B_Micro, J23 USB_A, J24 Conn_01x02_Male, J25 Barrel_Jack_Switch, J26 USB_B_Micro, J27 Conn_01x07_Male, J3 USB_B_Micro, J4 USB_B_Micro, J5 USB_B_Micro, J6 USB_B_Micro, J7 USB_B_Micro, J8 USB_B_Micro, J9 USB_B_Micro, SW1 SW_SPDT, U1 555, U2 74HC164, U3 4072, U4 74AHC1G04, U5 AP1117-33

Commit message: id
Parts:
- removed D134, D62, D66, D70, D75, D76: ledred, LED_SMD:LED_0603_1608Metric, symbol pace:ledred
- removed J14: USB_B_Micro, Connector_USB:USB_Micro-B_Molex-105017-0001, symbol pace:USB_B_Micro
- removed R29: 10k, Resistor_SMD:R_0402_1005Metric, symbol pace:10k
- removed TP74, TP79, TP80, TP86, TP90, TP94: TestPoint, TestPoint:TestPoint_Pad_D1.0mm, symbol pace:TestPoint
Changed lines of the file:
@@
 Connection ~ 5850 1400
-$Comp
-L pace:USB_B_Micro J14
-U 1 1 600595F2
-P 5450 2050
-F 0 "J14" H 5507 2425 50  0000 C CNN
-F 1 "USB_B_Micro" H 5250 2400 50  0001 L CNN
-F 2 "Connector_USB:USB_Micro-B_Molex-105017-0001" H 5600 2000 50  0001 C CNN
-F 3 "~" H 5600 2000 50  0001 C CNN
-	1    5450 2050
-	1    0    0    -1
-$EndComp
-$Comp
-L pace:TestPoint TP79
-U 1 1 600595F8
-P 5750 1850
-F 0 "TP79" H 5808 1922 50  0001 L CNN
-F 1 "TestPoint" H 5750 2050 50  0001 C CNN
-F 2 "TestPoint:TestPoint_Pad_D1.0mm" H 5950 1850 50  0001 C CNN
-F 3 "~" H 5950 1850 50  0001 C CNN
-	1    5750 1850
-	1    0    0    -1
-$EndComp
-$Comp
-L pace:ledred D62
-U 1 1 600595FF
-P 5850 1850
-F 0 "D62" H 5850 1750 50  0001 C CNN
-F 1 "ledred" H 5850 1994 50  0001 C CNN
-F 2 "LED_SMD:LED_0603_1608Metric" V 5850 1850 50  0001 C CNN
-F 3 "https://datasheet.lcsc.com/szlcsc/Hubei-KENTO-Elec-KT-0603R_C2286.pdf" V 5850 1850 50  0001 C CNN
-F 4 "C2286" H 5850 1850 50  0001 C CNN "LCSC"
-	1    5850 1850
-	-1   0    0    1
-$EndComp
-Connection ~ 5750 1850
-$Comp
-L pace:TestPoint TP90
-U 1 1 60059606
-P 5950 2050
-F 0 "TP90" H 6008 2122 50  0001 L CNN
-F 1 "TestPoint" H 5950 2250 50  0001 C CNN
-F 2 "TestPoint:TestPoint_Pad_D1.0mm" H 6150 2050 50  0001 C CNN
-F 3 "~" H 6150 2050 50  0001 C CNN
-	1    5950 2050
-	1    0    0    -1
-$EndComp
-$Comp
-L pace:ledred D70
-U 1 1 6005960D
-P 6050 2050
-F 0 "D70" H 6050 1950 50  0001 C CNN
-F 1 "ledred" H 6050 2194 50  0001 C CNN
-F 2 "LED_SMD:LED_0603_1608Metric" V 6050 2050 50  0001 C CNN
-F 3 "https://datasheet.lcsc.com/szlcsc/Hubei-KENTO-Elec-KT-0603R_C2286.pdf" V 6050 2050 50  0001 C CNN
-F 4 "C2286" H 6050 2050 50  0001 C CNN "LCSC"
-	1    6050 2050
-	-1   0    0    1
-$EndComp
-$Comp
-L pace:TestPoint TP94
-U 1 1 60059613
-P 6150 2150
-F 0 "TP94" H 6208 2222 50  0001 L CNN
-F 1 "TestPoint" H 6150 2350 50  0001 C CNN
-F 2 "TestPoint:TestPoint_Pad_D1.0mm" H 6350 2150 50  0001 C CNN
-F 3 "~" H 6350 2150 50  0001 C CNN
-	1    6150 2150
-	1    0    0    -1
-$EndComp
-$Comp
-L pace:ledred D75
-U 1 1 6005961A
-P 6250 2150
-F 0 "D75" H 6250 2050 50  0001 C CNN
-F 1 "ledred" H 6250 2294 50  0001 C CNN
-F 2 "LED_SMD:LED_0603_1608Metric" V 6250 2150 50  0001 C CNN
-F 3 "https://datasheet.lcsc.com/szlcsc/Hubei-KENTO-Elec-KT-0603R_C2286.pdf" V 6250 2150 50  0001 C CNN
-F 4 "C2286" H 6250 2150 50  0001 C CNN "LCSC"
-	1    6250 2150
-	-1   0    0    1
-$EndComp
-$Comp
-L pace:TestPoint TP80
-U 1 1 60059620
-P 6550 2250
-F 0 "TP80" H 6608 2322 50  0001 L CNN
-F 1 "TestPoint" H 6550 2450 50  0001 C CNN
-F 2 "TestPoint:TestPoint_Pad_D1.0mm" H 6750 2250 50  0001 C CNN
-F 3 "~" H 6750 2250 50  0001 C CNN
-	1    6550 2250
-	-1   0    0    1
-$EndComp
-$Comp
-L pace:TestPoint TP86
-U 1 1 60059626
-P 5850 2350
-F 0 "TP86" H 5908 2422 50  0001 L CNN
-F 1 "TestPoint" H 5850 2550 50  0001 C CNN
-F 2 "TestPoint:TestPoint_Pad_D1.0mm" H 6050 2350 50  0001 C CNN
-F 3 "~" H 6050 2350 50  0001 C CNN
-	1    5850 2350
-	1    0    0    -1
-$EndComp
-Wire Wire Line
-	5750 2050 5950 2050
-Connection ~ 5950 2050
-Connection ~ 6150 2150
-$Comp
-L pace:ledred D66
-U 1 1 60059633
-P 5950 2350
-F 0 "D66" H 5950 2250 50  0001 C CNN
-F 1 "ledred" H 5950 2494 50  0001 C CNN
-F 2 "LED_SMD:LED_0603_1608Metric" V 5950 2350 50  0001 C CNN
-F 3 "https://datasheet.lcsc.com/szlcsc/Hubei-KENTO-Elec-KT-0603R_C2286.pdf" V 5950 2350 50  0001 C CNN
-F 4 "C2286" H 5950 2350 50  0001 C CNN "LCSC"
-	1    5950 2350
-	-1   0    0    1
-$EndComp
-Wire Wire Line
-	5450 2450 5850 2450
-Wire Wire Line
-	5850 2450 5850 2350
-$Comp
-L pace:ledred D76
-U 1 1 6005963C
-P 6250 2500
-F 0 "D76" H 6250 2400 50  0001 C CNN
-F 1 "ledred" H 6250 2644 50  0001 C CNN
-F 2 "LED_SMD:LED_0603_1608Metric" V 6250 2500 50  0001 C CNN
-F 3 "https://datasheet.lcsc.com/szlcsc/Hubei-KENTO-Elec-KT-0603R_C2286.pdf" V 6250 2500 50  0001 C CNN
-F 4 "C2286" H 6250 2500 50  0001 C CNN "LCSC"
-	1    6250 2500
-	-1   0    0    1
-$EndComp
-Wire Wire Line
-	5350 2450 5350 2500
-Wire Wire Line
-	5350 2500 6150 2500
-$Comp
-L pace:TestPoint TP74
-U 1 1 60059644
-P 5350 2500
-F 0 "TP74" H 5408 2572 50  0001 L CNN
-F 1 "TestPoint" H 5350 2700 50  0001 C CNN
-F 2 "TestPoint:TestPoint_Pad_D1.0mm" H 5550 2500 50  0001 C CNN
-F 3 "~" H 5550 2500 50  0001 C CNN
-	1    5350 2500
-	0    -1   -1   0
-$EndComp
-Connection ~ 5350 2500
-$Comp
-L pace:GND #PWR?
-U 1 1 6005964B
-P 6350 2500
-F 0 "#PWR?" H 6350 2250 50  0001 C CNN
-F 1 "GND" H 6355 2327 50  0000 C CNN
-F 2 "" H 6350 2500 50  0001 C CNN
-F 3 "" H 6350 2500 50  0001 C CNN
-	1    6350 2500
-	1    0    0    -1
-$EndComp
-Wire Wire Line
-	5950 1850 6350 1850
-Wire Wire Line
-	6350 1850 6350 2050
-Connection ~ 6350 2500
-Connection ~ 6350 2150
-Wire Wire Line
-	6350 2150 6350 2350
-Wire Wire Line
-	6150 2050 6350 2050
-Connection ~ 6350 2050
-Wire Wire Line
-	6350 2050 6350 2150
-Wire Wire Line
-	6050 2350 6350 2350
-Connection ~ 6350 2350
-Wire Wire Line
-	6350 2350 6350 2500
-Connection ~ 5850 2350
 $Comp
 L pace:USB_B_Micro J15
@@
 	5750 1200 6150 1200
 Wire Wire Line
-	5750 2150 6150 2150
-Wire Wire Line
-	6550 2250 5750 2250
-Wire Wire Line
 	6550 1300 5750 1300
 Wire Wire Line
@@
 	1    0    0    -1
 $EndComp
-$Comp
-L pace:+3.3V #PWR?
-U 1 1 608F39EC
-P 6550 1850
-F 0 "#PWR?" H 6550 1700 50  0001 C CNN
-F 1 "+3.3V" H 6565 2023 50  0000 C CNN
-F 2 "" H 6550 1850 50  0001 C CNN
-F 3 "" H 6550 1850 50  0001 C CNN
-	1    6550 1850
-	1    0    0    -1
-$EndComp
-$Comp
-L pace:ledred D134
-U 1 1 608F39F3
-P 6550 1950
-F 0 "D134" H 6550 1850 50  0001 C CNN
-F 1 "ledred" H 6550 2094 50  0001 C CNN
-F 2 "LED_SMD:LED_0603_1608Metric" V 6550 1950 50  0001 C CNN
-F 3 "https://datasheet.lcsc.com/szlcsc/Hubei-KENTO-Elec-KT-0603R_C2286.pdf" V 6550 1950 50  0001 C CNN
-F 4 "C2286" H 6550 1950 50  0001 C CNN "LCSC"
-	1    6550 1950
-	0    -1   -1   0
-$EndComp
-$Comp
-L pace:10k R29
-U 1 1 608F39FA
-P 6550 2150
-F 0 "R29" V 6600 2300 50  0001 L CNN
-F 1 "10k" V 6600 1900 50  0001 L CNN
-F 2 "Resistor_SMD:R_0402_1005Metric" H 6550 2150 50  0001 C CNN
-F 3 "https://datasheet.lcsc.com/szlcsc/Uniroyal-Elec-0402WGF1002TCE_C25744.pdf" H 6550 2150 50  0001 C CNN
-F 4 "C25744" H 6550 2150 50  0001 C CNN "LCSC"
-	1    6550 2150
-	1    0    0    -1
-$EndComp

Commit message: routing
Parts:
- added C9: 100n, Capacitor_SMD:C_0402_1005Metric, symbol pace:100n
Connections:
- net +3V3: now also C9.1
- net GND: now also C9.2
- net at R3.1, U2.3 (Q0): now also U3.11; no longer U3.12
- net at R4.1, U2.4 (Q1): now also U3.10; no longer U3.11
- net at U3.1: now also U3.12; no longer U3.10
Changed lines of the file:
@@
 $Comp
 L pace:4072 U3
-U 1 1 601681B2
-P 5050 6000
-F 0 "U3" H 5050 6375 50  0000 C CNN
-F 1 "4072" H 5050 6284 50  0000 C CNN
-F 2 "Package_SO:SOIC-14_3.9x8.7mm_P1.27mm" H 5050 6000 50  0001 C CNN
-F 3 "http://www.intersil.com/content/dam/Intersil/documents/cd40/cd4071bms-72bms-75bms.pdf" H 5050 6000 50  0001 C CNN
-F 4 "C68527" H 5050 6000 50  0001 C CNN "LCSC"
-	1    5050 6000
-	1    0    0    -1
-$EndComp
-$Comp
-L pace:4072 U3
 U 2 1 601CB694
 P 5850 6300
@@
 	1    0    0    -1
 $EndComp
-Wire Wire Line
-	5350 6000 5450 6000
 NoConn ~ 4300 7450
 $Comp
@@
 Text GLabel 9700 6950 2    50   Input ~ 0
 TEST1
-Text Notes 8600 8100 0    50   ~ 0
+Text Notes 9050 8000 0    50   ~ 0
 pin 4 on the USB A connector\ngoes to pin 5 on the USB B
 Text GLabel 7850 7200 0    50   Input ~ 0
@@
 Wire Wire Line
 	4750 6150 4700 6150
-Wire Wire Line
-	5550 6350 5450 6350
 $Comp
 L pace:74AHC1G04 U4
@@
 	4300 7250 4500 7250
 Wire Wire Line
-	4300 7050 4700 7050
-Wire Wire Line
-	4300 6750 5550 6750
-Wire Wire Line
 	4300 7350 4400 7350
 Wire Wire Line
@@
 Wire Wire Line
 	4600 7150 5900 7150
-Wire Wire Line
-	4700 6150 4700 7050
-Connection ~ 4700 7050
-Wire Wire Line
-	4700 7050 5900 7050
-Wire Wire Line
-	4300 6950 5350 6950
-Wire Wire Line
-	4300 6850 5450 6850
-Connection ~ 5350 6950
-Wire Wire Line
-	5350 6950 5900 6950
-Wire Wire Line
-	5450 6350 5450 6850
-Connection ~ 5450 6850
-Wire Wire Line
-	5450 6850 5900 6850
-Wire Wire Line
-	5550 6450 5550 6750
-Connection ~ 5550 6750
-Wire Wire Line
-	5550 6750 5900 6750
-Wire Wire Line
-	5450 6000 5450 6250
-Wire Wire Line
-	5450 6250 5550 6250
-Wire Wire Line
-	5350 6150 5550 6150
-Wire Wire Line
-	5350 6150 5350 6950
 $Comp
 L pace:4072 U3
@@
 	1    0    0    -1
 $EndComp
+Wire Wire Line
+	4700 6150 4700 7050
+Wire Wire Line
+	4300 7050 4700 7050
+Connection ~ 4700 7050
+Wire Wire Line
+	4700 7050 5900 7050
+Wire Wire Line
+	5300 6850 5900 6850
+Wire Wire Line
+	4300 6850 5300 6850
+Connection ~ 5300 6850
+Wire Wire Line
+	5300 6250 5300 6850
+Wire Wire Line
+	5300 6250 5550 6250
+Wire Wire Line
+	5200 6950 5900 6950
+Wire Wire Line
+	4300 6950 5200 6950
+Connection ~ 5200 6950
+Wire Wire Line
+	5200 6150 5200 6950
+$Comp
+L pace:4072 U3
+U 1 1 601681B2
+P 5050 6000
+F 0 "U3" H 5050 6375 50  0000 C CNN
+F 1 "4072" H 5050 6284 50  0000 C CNN
+F 2 "Package_SO:SOIC-14_3.9x8.7mm_P1.27mm" H 5050 6000 50  0001 C CNN
+F 3 "http://www.intersil.com/content/dam/Intersil/documents/cd40/cd4071bms-72bms-75bms.pdf" H 5050 6000 50  0001 C CNN
+F 4 "C68527" H 5050 6000 50  0001 C CNN "LCSC"
+	1    5050 6000
+	1    0    0    -1
+$EndComp
+Wire Wire Line
+	5200 6150 5550 6150
+Wire Wire Line
+	4300 6750 5400 6750
+Wire Wire Line
+	5550 6350 5400 6350
+Wire Wire Line
+	5400 6350 5400 6750
+Connection ~ 5400 6750
+Wire Wire Line
+	5400 6750 5900 6750
+Wire Wire Line
+	5350 6000 5500 6000
+Wire Wire Line
+	5500 6000 5500 6450
+Wire Wire Line
+	5500 6450 5550 6450
+$Comp
+L pace:100n C9
+U 1 1 604E3FC4
+P 8550 7900
+F 0 "C9" H 8642 7946 50  0000 L CNN
+F 1 "100n" H 8642 7855 50  0000 L CNN
+F 2 "Capacitor_SMD:C_0402_1005Metric" H 8550 7900 50  0001 C CNN
+F 3 "https://datasheet.lcsc.com/szlcsc/Samsung-Electro-Mechanics-CL05B104KO5NNNC_C1525.pdf" H 8550 7900 50  0001 C CNN
+F 4 "C1525" H 8550 7900 50  0001 C CNN "LCSC"
+	1    8550 7900
+	1    0    0    -1
+$EndComp
+Wire Wire Line
+	8200 8000 8550 8000
+Connection ~ 8200 8000
+Wire Wire Line
+	8200 7800 8550 7800
+Connection ~ 8200 7800
 $EndSCHEMATC

Commit message: fab
Parts:
- U4: LCSC (none) -> C7466
Changed lines of the file:
@@
 F 2 "Package_TO_SOT_SMD:SOT-353_SC-70-5" H 6650 6300 50  0001 C CNN
 F 3 "https://lcsc.com/product-detail/74-Series_TI_SN74AHC1G04DCKR_SN74AHC1G04DCKR_C7466.html/?href=jlc-SMT" H 6650 6300 50  0001 C CNN
+F 4 "C7466" H 6650 6300 50  0001 C CNN "LCSC"
 	1    6650 6300
 	1    0    0    -1
